File: hw/skylark-usb/boards/skylark-usb/03_ADC_reference-page-02.kicad_sch (KiCad schematic)
At the start: 8 parts, among them U5 OPA387DBVR, U6 ADS122C04IPWR

Commit message: Harden Skylark signal chain and add manufacturing audit
Parts:
- R71: value 1e+06R -> 100000R; MPN RC0603FR-071ML -> RT0603BRD07100KL
Connections:
- net GND: no longer R71.2
- net VZERO: now also R71.2
- net USB_5V renamed GATE_SUPPLY
Changed lines of the file:
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@@
               (instances (project "skylark-usb" (path "/dafe1df7-5e39-58a9-9d86-b1c10fa6f345/e7f2d07d-a3bf-5eff-bec3-079d79795f18" (reference "R70") (unit 1)))))
 (wire (pts (xy 223.52 83.82) (xy 218.44 83.82)) (stroke (width 0) (type default)))
-(global_label "USB_5V" (shape bidirectional) (at 218.44 83.82 180) (effects (font (size 0.9 0.9)) (justify right)))
+(global_label "GATE_SUPPLY" (shape bidirectional) (at 218.44 83.82 180) (effects (font (size 0.9 0.9)) (justify right)))
 (wire (pts (xy 254.0 83.82) (xy 259.08 83.82)) (stroke (width 0) (type default)))
 (global_label "CLAMP_GATE" (shape bidirectional) (at 259.08 83.82 0) (effects (font (size 0.9 0.9)) (justify left)))
 (symbol (lib_id "Groundlark:Part_R71") (at 335.28 83.82000000000001 0) (unit 1) (in_bom yes) (on_board yes) (dnp no)
               (property "Reference" "R71" (at 335.28 77.28 0) (effects (font (size 1.27 1.27))))
-              (property "Value" "1e+06R" (at 335.28 79.78 0) (effects (font (size 1.0 1.0))))
+              (property "Value" "100000R" (at 335.28 79.78 0) (effects (font (size 1.0 1.0))))
               (property "Footprint" "Skylark:Resistor_SMD__R_0603_1608Metric" (at 335.28 83.82000000000001 0) (effects (font (size 1 1)) hide))
-              (property "MPN" "RC0603FR-071ML" (at 335.28 83.82000000000001 0) (effects (font (size 1 1)) hide))
+              (property "MPN" "RT0603BRD07100KL" (at 335.28 83.82000000000001 0) (effects (font (size 1 1)) hide))
               (instances (project "skylark-usb" (path "/dafe1df7-5e39-58a9-9d86-b1c10fa6f345/e7f2d07d-a3bf-5eff-bec3-079d79795f18" (reference "R71") (unit 1)))))
 (wire (pts (xy 320.04 83.82) (xy 314.96 83.82)) (stroke (width 0) (type default)))
 (global_label "CLAMP_GATE" (shape bidirectional) (at 314.96 83.82 180) (effects (font (size 0.9 0.9)) (justify right)))
 (wire (pts (xy 350.52 83.82) (xy 355.6 83.82)) (stroke (width 0) (type default)))
-(global_label "GND" (shape bidirectional) (at 355.6 83.82 0) (effects (font (size 0.9 0.9)) (justify left)))
+(global_label "VZERO" (shape bidirectional) (at 355.6 83.82 0) (effects (font (size 0.9 0.9)) (justify left)))
 )
