File: hw/skylark-usb/boards/skylark-usb/04_Analog_reference-page-01.kicad_sch (KiCad schematic)
At the start: 6 parts, among them Q7 2N7002/HAMR, U13 TPS22918DBVR

Commit message: Harden Skylark signal chain and add manufacturing audit
Parts:
- added D4: BAT54LT1G, Skylark:Package_TO_SOT_SMD__SOT-23, symbol Groundlark:Part_D4
- added R74: 10000R, Skylark:Resistor_SMD__R_0603_1608Metric, symbol Groundlark:Part_R74
- Q7: value 2N7002/HAMR -> MMBT3904LT1G; MPN 2N7002/HAMR -> MMBT3904LT1G
Connections:
- net CLAMP_HOLD: now also R74.1; no longer Q7.1 (G)
- net GND: no longer Q7.2 (S)
- new net CLAMP_BASE: Q7.1 (G), R74.2
- new net GATE_SUPPLY: D4.3 (D)
- new net USB_5V: D4.1 (G)
- new net VZERO: Q7.2 (S)
- no-connect marks 0 -> 1
Changed lines of the file:
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@@
 (symbol (lib_id "Groundlark:Part_Q7") (at 142.24 39.370000000000005 0) (unit 1) (in_bom yes) (on_board yes) (dnp no)
               (property "Reference" "Q7" (at 142.24 31.560000000000002 0) (effects (font (size 1.27 1.27))))
-              (property "Value" "2N7002/HAMR" (at 142.24 34.06 0) (effects (font (size 1.0 1.0))))
+              (property "Value" "MMBT3904LT1G" (at 142.24 34.06 0) (effects (font (size 1.0 1.0))))
               (property "Footprint" "Skylark:Package_TO_SOT_SMD__SOT-23" (at 142.24 39.370000000000005 0) (effects (font (size 1 1)) hide))
-              (property "MPN" "2N7002/HAMR" (at 142.24 39.370000000000005 0) (effects (font (size 1 1)) hide))
+              (property "MPN" "MMBT3904LT1G" (at 142.24 39.370000000000005 0) (effects (font (size 1 1)) hide))
               (instances (project "skylark-usb" (path "/dafe1df7-5e39-58a9-9d86-b1c10fa6f345/355762cb-5426-5567-9d3e-d33b6f259b0a" (reference "Q7") (unit 1)))))
 (wire (pts (xy 127.0 38.1) (xy 121.92 38.1)) (stroke (width 0) (type default)))
-(global_label "CLAMP_HOLD" (shape bidirectional) (at 121.92 38.1 180) (effects (font (size 0.9 0.9)) (justify right)))
+(global_label "CLAMP_BASE" (shape bidirectional) (at 121.92 38.1 180) (effects (font (size 0.9 0.9)) (justify right)))
 (wire (pts (xy 127.0 40.64) (xy 121.92 40.64)) (stroke (width 0) (type default)))
-(global_label "GND" (shape bidirectional) (at 121.92 40.64 180) (effects (font (size 0.9 0.9)) (justify right)))
+(global_label "VZERO" (shape bidirectional) (at 121.92 40.64 180) (effects (font (size 0.9 0.9)) (justify right)))
 (wire (pts (xy 157.48 38.1) (xy 162.56 38.1)) (stroke (width 0) (type default)))
 (global_label "CLAMP_GATE" (shape bidirectional) (at 162.56 38.1 0) (effects (font (size 0.9 0.9)) (justify left)))
@@
 (wire (pts (xy 157.48 71.12) (xy 162.56 71.12)) (stroke (width 0) (type default)))
 (global_label "GND" (shape bidirectional) (at 162.56 71.12 0) (effects (font (size 0.9 0.9)) (justify left)))
+(symbol (lib_id "Groundlark:Part_R74") (at 238.76 71.12 0) (unit 1) (in_bom yes) (on_board yes) (dnp no)
+              (property "Reference" "R74" (at 238.76 64.58 0) (effects (font (size 1.27 1.27))))
+              (property "Value" "10000R" (at 238.76 67.08 0) (effects (font (size 1.0 1.0))))
+              (property "Footprint" "Skylark:Resistor_SMD__R_0603_1608Metric" (at 238.76 71.12 0) (effects (font (size 1 1)) hide))
+              (property "MPN" "RT0603BRD0710KL" (at 238.76 71.12 0) (effects (font (size 1 1)) hide))
+              (instances (project "skylark-usb" (path "/dafe1df7-5e39-58a9-9d86-b1c10fa6f345/355762cb-5426-5567-9d3e-d33b6f259b0a" (reference "R74") (unit 1)))))
+(wire (pts (xy 223.52 71.12) (xy 218.44 71.12)) (stroke (width 0) (type default)))
+(global_label "CLAMP_HOLD" (shape bidirectional) (at 218.44 71.12 180) (effects (font (size 0.9 0.9)) (justify right)))
+(wire (pts (xy 254.0 71.12) (xy 259.08 71.12)) (stroke (width 0) (type default)))
+(global_label "CLAMP_BASE" (shape bidirectional) (at 259.08 71.12 0) (effects (font (size 0.9 0.9)) (justify left)))
+(symbol (lib_id "Groundlark:Part_D4") (at 335.28 72.39 0) (unit 1) (in_bom yes) (on_board yes) (dnp no)
+              (property "Reference" "D4" (at 335.28 64.58 0) (effects (font (size 1.27 1.27))))
+              (property "Value" "BAT54LT1G" (at 335.28 67.08 0) (effects (font (size 1.0 1.0))))
+              (property "Footprint" "Skylark:Package_TO_SOT_SMD__SOT-23" (at 335.28 72.39 0) (effects (font (size 1 1)) hide))
+              (property "MPN" "BAT54LT1G" (at 335.28 72.39 0) (effects (font (size 1 1)) hide))
+              (instances (project "skylark-usb" (path "/dafe1df7-5e39-58a9-9d86-b1c10fa6f345/355762cb-5426-5567-9d3e-d33b6f259b0a" (reference "D4") (unit 1)))))
+(wire (pts (xy 320.04 71.12) (xy 314.96 71.12)) (stroke (width 0) (type default)))
+(global_label "USB_5V" (shape bidirectional) (at 314.96 71.12 180) (effects (font (size 0.9 0.9)) (justify right)))
+(no_connect (at 320.04 73.66))
+(wire (pts (xy 350.52 71.12) (xy 355.6 71.12)) (stroke (width 0) (type default)))
+(global_label "GATE_SUPPLY" (shape bidirectional) (at 355.6 71.12 0) (effects (font (size 0.9 0.9)) (justify left)))
 )
