File: hw/skylark-usb/boards/skylark-usb/01_USB_power-page-01.kicad_sch (KiCad schematic)
At the start: 12 parts, among them J1 USB4105-GF-A, U2 AP2112K-3.3TRG1, U3 TPS2553DBVR

Commit message: Finalize Skylark signal-chain updates and remove obsolete artifacts
Parts:
- J1: value USB4105-GF-A -> TYPE-C-31-M-12; footprint Skylark:Connector_USB__USB_C_Receptacle_GCT_USB4105-xx-A_16P_TopMnt_Horizontal -> Skylark:USB_C_HRO_TYPE-C-31-M-12; MPN USB4105-GF-A -> TYPE-C-31-M-12
- R3: value 80600R -> 82000R; MPN RC0603FR-0780K6L -> RC0603FR-0782KL
Connections:
- net GND: now also J1.A1B12, J1.B1A12; no longer J1.A1, J1.A12, J1.B1, J1.B12
- net USB_VBUS: now also J1.A4B9, J1.B4A9; no longer J1.A4, J1.A9, J1.B4, J1.B9
Other:
- moved on the sheet: C1, C2, D2, F1, R3, R4, U2, U3
