File: hw/skylark-usb/boards/skylark-usb/04_SO2-page-02.kicad_sch (KiCad schematic)
At the start: 8 parts, among them Q2 MMBFJ177LT1G

Commit message: Harden Skylark signal chain and add manufacturing audit
Parts:
- added R75: 100R, Skylark:Resistor_SMD__R_0603_1608Metric, symbol Groundlark:Part_R75
- C36: footprint Skylark:Capacitor_SMD__C_0603_1608Metric -> Skylark:Capacitor_SMD__C_1206_3216Metric; MPN GRM188R71H104KA93D -> C3216C0G1H104JT000N
- Q2: value MMBFJ177LT1G -> MMBFJ270; MPN MMBFJ177LT1G -> MMBFJ270
Connections:
- new net VZERO: R75.1
- no-connect marks 0 -> 1
Changed lines of the file:
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@@
 (symbol (lib_id "Groundlark:Part_Q2") (at 238.76 39.370000000000005 0) (unit 1) (in_bom yes) (on_board yes) (dnp no)
               (property "Reference" "Q2" (at 238.76 31.560000000000002 0) (effects (font (size 1.27 1.27))))
-              (property "Value" "MMBFJ177LT1G" (at 238.76 34.06 0) (effects (font (size 1.0 1.0))))
+              (property "Value" "MMBFJ270" (at 238.76 34.06 0) (effects (font (size 1.0 1.0))))
               (property "Footprint" "Skylark:Package_TO_SOT_SMD__SOT-23" (at 238.76 39.370000000000005 0) (effects (font (size 1 1)) hide))
-              (property "MPN" "MMBFJ177LT1G" (at 238.76 39.370000000000005 0) (effects (font (size 1 1)) hide))
+              (property "MPN" "MMBFJ270" (at 238.76 39.370000000000005 0) (effects (font (size 1 1)) hide))
               (instances (project "skylark-usb" (path "/dafe1df7-5e39-58a9-9d86-b1c10fa6f345/fba23098-6c42-5f5d-abd6-c7297354137a" (reference "Q2") (unit 1)))))
 (wire (pts (xy 223.52 38.1) (xy 218.44 38.1)) (stroke (width 0) (type default)))
@@
               (property "Reference" "C36" (at 142.24 62.040000000000006 0) (effects (font (size 1.27 1.27))))
               (property "Value" "100nF" (at 142.24 64.54 0) (effects (font (size 1.0 1.0))))
-              (property "Footprint" "Skylark:Capacitor_SMD__C_0603_1608Metric" (at 142.24 68.58000000000001 0) (effects (font (size 1 1)) hide))
-              (property "MPN" "GRM188R71H104KA93D" (at 142.24 68.58000000000001 0) (effects (font (size 1 1)) hide))
+              (property "Footprint" "Skylark:Capacitor_SMD__C_1206_3216Metric" (at 142.24 68.58000000000001 0) (effects (font (size 1 1)) hide))
+              (property "MPN" "C3216C0G1H104JT000N" (at 142.24 68.58000000000001 0) (effects (font (size 1 1)) hide))
               (instances (project "skylark-usb" (path "/dafe1df7-5e39-58a9-9d86-b1c10fa6f345/fba23098-6c42-5f5d-abd6-c7297354137a" (reference "C36") (unit 1)))))
 (wire (pts (xy 127.0 68.58) (xy 121.92 68.58)) (stroke (width 0) (type default)))
@@
 (wire (pts (xy 350.52 68.58) (xy 355.6 68.58)) (stroke (width 0) (type default)))
 (global_label "GND" (shape bidirectional) (at 355.6 68.58 0) (effects (font (size 0.9 0.9)) (justify left)))
+(symbol (lib_id "Groundlark:Part_R75") (at 45.72 96.52000000000001 0) (unit 1) (in_bom yes) (on_board yes) (dnp no)
+              (property "Reference" "R75" (at 45.72 89.98 0) (effects (font (size 1.27 1.27))))
+              (property "Value" "100R" (at 45.72 92.48 0) (effects (font (size 1.0 1.0))))
+              (property "Footprint" "Skylark:Resistor_SMD__R_0603_1608Metric" (at 45.72 96.52000000000001 0) (effects (font (size 1 1)) hide))
+              (property "MPN" "RC0603FR-07100RL" (at 45.72 96.52000000000001 0) (effects (font (size 1 1)) hide))
+              (instances (project "skylark-usb" (path "/dafe1df7-5e39-58a9-9d86-b1c10fa6f345/fba23098-6c42-5f5d-abd6-c7297354137a" (reference "R75") (unit 1)))))
+(wire (pts (xy 30.48 96.52) (xy 25.4 96.52)) (stroke (width 0) (type default)))
+(global_label "VZERO" (shape bidirectional) (at 25.4 96.52 180) (effects (font (size 0.9 0.9)) (justify right)))
+(no_connect (at 60.96 96.52))
 )

Commit message: Finalize Skylark signal-chain updates and remove obsolete artifacts
Parts:
- C34: value 1uF -> 10uF; footprint Skylark:Capacitor_SMD__C_0603_1608Metric -> Skylark:Capacitor_SMD__C_0805_2012Metric; MPN GRM188R71E105KA12D -> GRM21BR61A106KE19L
Changed lines of the file:
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@@
 (symbol (lib_id "Groundlark:Part_C34") (at 142.24 38.1 0) (unit 1) (in_bom yes) (on_board yes) (dnp no)
               (property "Reference" "C34" (at 142.24 31.560000000000002 0) (effects (font (size 1.27 1.27))))
-              (property "Value" "1uF" (at 142.24 34.06 0) (effects (font (size 1.0 1.0))))
-              (property "Footprint" "Skylark:Capacitor_SMD__C_0603_1608Metric" (at 142.24 38.1 0) (effects (font (size 1 1)) hide))
-              (property "MPN" "GRM188R71E105KA12D" (at 142.24 38.1 0) (effects (font (size 1 1)) hide))
+              (property "Value" "10uF" (at 142.24 34.06 0) (effects (font (size 1.0 1.0))))
+              (property "Footprint" "Skylark:Capacitor_SMD__C_0805_2012Metric" (at 142.24 38.1 0) (effects (font (size 1 1)) hide))
+              (property "MPN" "GRM21BR61A106KE19L" (at 142.24 38.1 0) (effects (font (size 1 1)) hide))
               (instances (project "skylark-usb" (path "/dafe1df7-5e39-58a9-9d86-b1c10fa6f345/fba23098-6c42-5f5d-abd6-c7297354137a" (reference "C34") (unit 1)))))
 (wire (pts (xy 127.0 38.1) (xy 121.92 38.1)) (stroke (width 0) (type default)))
