File: hw/skylark-usb/boards/skylark-usb/05_H2S-page-01.kicad_sch (KiCad schematic)
At the start: 12 parts, among them Q3 MMBFJ177LT1G, U10 OPA387DBVR, U9 OPA2387DGKR

Commit message: Harden Skylark signal chain and add manufacturing audit
Parts:
- C50, C53: value 470nF -> 100nF; footprint Skylark:Capacitor_SMD__C_0603_1608Metric -> Skylark:Capacitor_SMD__C_1206_3216Metric; MPN GRM188R71E474KA12D -> C3216C0G1H104JT000N
- Q3: value MMBFJ177LT1G -> MMBFJ270; MPN MMBFJ177LT1G -> MMBFJ270
Changed lines of the file:
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@@
 (symbol (lib_id "Groundlark:Part_C50") (at 142.24 73.66000000000001 0) (unit 1) (in_bom yes) (on_board yes) (dnp no)
               (property "Reference" "C50" (at 142.24 67.12 0) (effects (font (size 1.27 1.27))))
-              (property "Value" "470nF" (at 142.24 69.62 0) (effects (font (size 1.0 1.0))))
-              (property "Footprint" "Skylark:Capacitor_SMD__C_0603_1608Metric" (at 142.24 73.66000000000001 0) (effects (font (size 1 1)) hide))
-              (property "MPN" "GRM188R71E474KA12D" (at 142.24 73.66000000000001 0) (effects (font (size 1 1)) hide))
+              (property "Value" "100nF" (at 142.24 69.62 0) (effects (font (size 1.0 1.0))))
+              (property "Footprint" "Skylark:Capacitor_SMD__C_1206_3216Metric" (at 142.24 73.66000000000001 0) (effects (font (size 1 1)) hide))
+              (property "MPN" "C3216C0G1H104JT000N" (at 142.24 73.66000000000001 0) (effects (font (size 1 1)) hide))
               (instances (project "skylark-usb" (path "/dafe1df7-5e39-58a9-9d86-b1c10fa6f345/ff6b77c3-95f8-5afc-8a6a-99a7ff58b4d5" (reference "C50") (unit 1)))))
 (wire (pts (xy 127.0 73.66) (xy 121.92 73.66)) (stroke (width 0) (type default)))
@@
 (symbol (lib_id "Groundlark:Part_Q3") (at 45.72 102.87 0) (unit 1) (in_bom yes) (on_board yes) (dnp no)
               (property "Reference" "Q3" (at 45.72 95.06 0) (effects (font (size 1.27 1.27))))
-              (property "Value" "MMBFJ177LT1G" (at 45.72 97.56 0) (effects (font (size 1.0 1.0))))
+              (property "Value" "MMBFJ270" (at 45.72 97.56 0) (effects (font (size 1.0 1.0))))
               (property "Footprint" "Skylark:Package_TO_SOT_SMD__SOT-23" (at 45.72 102.87 0) (effects (font (size 1 1)) hide))
-              (property "MPN" "MMBFJ177LT1G" (at 45.72 102.87 0) (effects (font (size 1 1)) hide))
+              (property "MPN" "MMBFJ270" (at 45.72 102.87 0) (effects (font (size 1 1)) hide))
               (instances (project "skylark-usb" (path "/dafe1df7-5e39-58a9-9d86-b1c10fa6f345/ff6b77c3-95f8-5afc-8a6a-99a7ff58b4d5" (reference "Q3") (unit 1)))))
 (wire (pts (xy 30.48 101.6) (xy 25.4 101.6)) (stroke (width 0) (type default)))
@@
 (symbol (lib_id "Groundlark:Part_C53") (at 335.28 101.60000000000001 0) (unit 1) (in_bom yes) (on_board yes) (dnp no)
               (property "Reference" "C53" (at 335.28 95.06 0) (effects (font (size 1.27 1.27))))
-              (property "Value" "470nF" (at 335.28 97.56 0) (effects (font (size 1.0 1.0))))
-              (property "Footprint" "Skylark:Capacitor_SMD__C_0603_1608Metric" (at 335.28 101.60000000000001 0) (effects (font (size 1 1)) hide))
-              (property "MPN" "GRM188R71E474KA12D" (at 335.28 101.60000000000001 0) (effects (font (size 1 1)) hide))
+              (property "Value" "100nF" (at 335.28 97.56 0) (effects (font (size 1.0 1.0))))
+              (property "Footprint" "Skylark:Capacitor_SMD__C_1206_3216Metric" (at 335.28 101.60000000000001 0) (effects (font (size 1 1)) hide))
+              (property "MPN" "C3216C0G1H104JT000N" (at 335.28 101.60000000000001 0) (effects (font (size 1 1)) hide))
               (instances (project "skylark-usb" (path "/dafe1df7-5e39-58a9-9d86-b1c10fa6f345/ff6b77c3-95f8-5afc-8a6a-99a7ff58b4d5" (reference "C53") (unit 1)))))
 (wire (pts (xy 320.04 101.6) (xy 314.96 101.6)) (stroke (width 0) (type default)))

Commit message: Finalize Skylark signal-chain updates and remove obsolete artifacts
Parts:
- C51: value 1uF -> 10uF; footprint Skylark:Capacitor_SMD__C_0603_1608Metric -> Skylark:Capacitor_SMD__C_0805_2012Metric; MPN GRM188R71E105KA12D -> GRM21BR61A106KE19L
Changed lines of the file:
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@@
 (symbol (lib_id "Groundlark:Part_C51") (at 335.28 73.66000000000001 0) (unit 1) (in_bom yes) (on_board yes) (dnp no)
               (property "Reference" "C51" (at 335.28 67.12 0) (effects (font (size 1.27 1.27))))
-              (property "Value" "1uF" (at 335.28 69.62 0) (effects (font (size 1.0 1.0))))
-              (property "Footprint" "Skylark:Capacitor_SMD__C_0603_1608Metric" (at 335.28 73.66000000000001 0) (effects (font (size 1 1)) hide))
-              (property "MPN" "GRM188R71E105KA12D" (at 335.28 73.66000000000001 0) (effects (font (size 1 1)) hide))
+              (property "Value" "10uF" (at 335.28 69.62 0) (effects (font (size 1.0 1.0))))
+              (property "Footprint" "Skylark:Capacitor_SMD__C_0805_2012Metric" (at 335.28 73.66000000000001 0) (effects (font (size 1 1)) hide))
+              (property "MPN" "GRM21BR61A106KE19L" (at 335.28 73.66000000000001 0) (effects (font (size 1 1)) hide))
               (instances (project "skylark-usb" (path "/dafe1df7-5e39-58a9-9d86-b1c10fa6f345/ff6b77c3-95f8-5afc-8a6a-99a7ff58b4d5" (reference "C51") (unit 1)))))
 (wire (pts (xy 320.04 73.66) (xy 314.96 73.66)) (stroke (width 0) (type default)))
