File: hw/skylark-usb/boards/skylark-usb/05_H2S-page-02.kicad_sch (KiCad schematic)
At the start: 8 parts, among them Q4 MMBFJ177LT1G

Commit message: Harden Skylark signal chain and add manufacturing audit
Parts:
- added C80: 100nF, Skylark:Capacitor_SMD__C_1206_3216Metric, symbol Groundlark:Part_C80
- added C81: 100nF, Skylark:Capacitor_SMD__C_1206_3216Metric, symbol Groundlark:Part_C81
- added C82: 100nF, Skylark:Capacitor_SMD__C_1206_3216Metric, symbol Groundlark:Part_C82
- added C83: 100nF, Skylark:Capacitor_SMD__C_1206_3216Metric, symbol Groundlark:Part_C83
- C56: footprint Skylark:Capacitor_SMD__C_0603_1608Metric -> Skylark:Capacitor_SMD__C_1206_3216Metric; MPN GRM188R71H104KA93D -> C3216C0G1H104JT000N
- Q4: value MMBFJ177LT1G -> MMBFJ270; MPN MMBFJ177LT1G -> MMBFJ270
Connections:
- new net H2S_WE_OUT: C80.2, C81.2, C82.2, C83.2
- new net H2S_WE_SUM: C80.1, C81.1, C82.1, C83.1
Changed lines of the file:
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@@
 (symbol (lib_id "Groundlark:Part_Q4") (at 238.76 39.370000000000005 0) (unit 1) (in_bom yes) (on_board yes) (dnp no)
               (property "Reference" "Q4" (at 238.76 31.560000000000002 0) (effects (font (size 1.27 1.27))))
-              (property "Value" "MMBFJ177LT1G" (at 238.76 34.06 0) (effects (font (size 1.0 1.0))))
+              (property "Value" "MMBFJ270" (at 238.76 34.06 0) (effects (font (size 1.0 1.0))))
               (property "Footprint" "Skylark:Package_TO_SOT_SMD__SOT-23" (at 238.76 39.370000000000005 0) (effects (font (size 1 1)) hide))
-              (property "MPN" "MMBFJ177LT1G" (at 238.76 39.370000000000005 0) (effects (font (size 1 1)) hide))
+              (property "MPN" "MMBFJ270" (at 238.76 39.370000000000005 0) (effects (font (size 1 1)) hide))
               (instances (project "skylark-usb" (path "/dafe1df7-5e39-58a9-9d86-b1c10fa6f345/c60510a4-912f-56f4-a510-e17dcca6cdbf" (reference "Q4") (unit 1)))))
 (wire (pts (xy 223.52 38.1) (xy 218.44 38.1)) (stroke (width 0) (type default)))
@@
               (property "Reference" "C56" (at 142.24 62.040000000000006 0) (effects (font (size 1.27 1.27))))
               (property "Value" "100nF" (at 142.24 64.54 0) (effects (font (size 1.0 1.0))))
-              (property "Footprint" "Skylark:Capacitor_SMD__C_0603_1608Metric" (at 142.24 68.58000000000001 0) (effects (font (size 1 1)) hide))
-              (property "MPN" "GRM188R71H104KA93D" (at 142.24 68.58000000000001 0) (effects (font (size 1 1)) hide))
+              (property "Footprint" "Skylark:Capacitor_SMD__C_1206_3216Metric" (at 142.24 68.58000000000001 0) (effects (font (size 1 1)) hide))
+              (property "MPN" "C3216C0G1H104JT000N" (at 142.24 68.58000000000001 0) (effects (font (size 1 1)) hide))
               (instances (project "skylark-usb" (path "/dafe1df7-5e39-58a9-9d86-b1c10fa6f345/c60510a4-912f-56f4-a510-e17dcca6cdbf" (reference "C56") (unit 1)))))
 (wire (pts (xy 127.0 68.58) (xy 121.92 68.58)) (stroke (width 0) (type default)))
@@
 (wire (pts (xy 350.52 68.58) (xy 355.6 68.58)) (stroke (width 0) (type default)))
 (global_label "GND" (shape bidirectional) (at 355.6 68.58 0) (effects (font (size 0.9 0.9)) (justify left)))
+(symbol (lib_id "Groundlark:Part_C80") (at 45.72 96.52000000000001 0) (unit 1) (in_bom yes) (on_board yes) (dnp no)
+              (property "Reference" "C80" (at 45.72 89.98 0) (effects (font (size 1.27 1.27))))
+              (property "Value" "100nF" (at 45.72 92.48 0) (effects (font (size 1.0 1.0))))
+              (property "Footprint" "Skylark:Capacitor_SMD__C_1206_3216Metric" (at 45.72 96.52000000000001 0) (effects (font (size 1 1)) hide))
+              (property "MPN" "C3216C0G1H104JT000N" (at 45.72 96.52000000000001 0) (effects (font (size 1 1)) hide))
+              (instances (project "skylark-usb" (path "/dafe1df7-5e39-58a9-9d86-b1c10fa6f345/c60510a4-912f-56f4-a510-e17dcca6cdbf" (reference "C80") (unit 1)))))
+(wire (pts (xy 30.48 96.52) (xy 25.4 96.52)) (stroke (width 0) (type default)))
+(global_label "H2S_WE_SUM" (shape bidirectional) (at 25.4 96.52 180) (effects (font (size 0.9 0.9)) (justify right)))
+(wire (pts (xy 60.96 96.52) (xy 66.04 96.52)) (stroke (width 0) (type default)))
+(global_label "H2S_WE_OUT" (shape bidirectional) (at 66.04 96.52 0) (effects (font (size 0.9 0.9)) (justify left)))
+(symbol (lib_id "Groundlark:Part_C81") (at 142.24 96.52000000000001 0) (unit 1) (in_bom yes) (on_board yes) (dnp no)
+              (property "Reference" "C81" (at 142.24 89.98 0) (effects (font (size 1.27 1.27))))
+              (property "Value" "100nF" (at 142.24 92.48 0) (effects (font (size 1.0 1.0))))
+              (property "Footprint" "Skylark:Capacitor_SMD__C_1206_3216Metric" (at 142.24 96.52000000000001 0) (effects (font (size 1 1)) hide))
+              (property "MPN" "C3216C0G1H104JT000N" (at 142.24 96.52000000000001 0) (effects (font (size 1 1)) hide))
+              (instances (project "skylark-usb" (path "/dafe1df7-5e39-58a9-9d86-b1c10fa6f345/c60510a4-912f-56f4-a510-e17dcca6cdbf" (reference "C81") (unit 1)))))
+(wire (pts (xy 127.0 96.52) (xy 121.92 96.52)) (stroke (width 0) (type default)))
+(global_label "H2S_WE_SUM" (shape bidirectional) (at 121.92 96.52 180) (effects (font (size 0.9 0.9)) (justify right)))
+(wire (pts (xy 157.48 96.52) (xy 162.56 96.52)) (stroke (width 0) (type default)))
+(global_label "H2S_WE_OUT" (shape bidirectional) (at 162.56 96.52 0) (effects (font (size 0.9 0.9)) (justify left)))
+(symbol (lib_id "Groundlark:Part_C82") (at 238.76 96.52000000000001 0) (unit 1) (in_bom yes) (on_board yes) (dnp no)
+              (property "Reference" "C82" (at 238.76 89.98 0) (effects (font (size 1.27 1.27))))
+              (property "Value" "100nF" (at 238.76 92.48 0) (effects (font (size 1.0 1.0))))
+              (property "Footprint" "Skylark:Capacitor_SMD__C_1206_3216Metric" (at 238.76 96.52000000000001 0) (effects (font (size 1 1)) hide))
+              (property "MPN" "C3216C0G1H104JT000N" (at 238.76 96.52000000000001 0) (effects (font (size 1 1)) hide))
+              (instances (project "skylark-usb" (path "/dafe1df7-5e39-58a9-9d86-b1c10fa6f345/c60510a4-912f-56f4-a510-e17dcca6cdbf" (reference "C82") (unit 1)))))
+(wire (pts (xy 223.52 96.52) (xy 218.44 96.52)) (stroke (width 0) (type default)))
+(global_label "H2S_WE_SUM" (shape bidirectional) (at 218.44 96.52 180) (effects (font (size 0.9 0.9)) (justify right)))
+(wire (pts (xy 254.0 96.52) (xy 259.08 96.52)) (stroke (width 0) (type default)))
+(global_label "H2S_WE_OUT" (shape bidirectional) (at 259.08 96.52 0) (effects (font (size 0.9 0.9)) (justify left)))
+(symbol (lib_id "Groundlark:Part_C83") (at 335.28 96.52000000000001 0) (unit 1) (in_bom yes) (on_board yes) (dnp no)
+              (property "Reference" "C83" (at 335.28 89.98 0) (effects (font (size 1.27 1.27))))
+              (property "Value" "100nF" (at 335.28 92.48 0) (effects (font (size 1.0 1.0))))
+              (property "Footprint" "Skylark:Capacitor_SMD__C_1206_3216Metric" (at 335.28 96.52000000000001 0) (effects (font (size 1 1)) hide))
+              (property "MPN" "C3216C0G1H104JT000N" (at 335.28 96.52000000000001 0) (effects (font (size 1 1)) hide))
+              (instances (project "skylark-usb" (path "/dafe1df7-5e39-58a9-9d86-b1c10fa6f345/c60510a4-912f-56f4-a510-e17dcca6cdbf" (reference "C83") (unit 1)))))
+(wire (pts (xy 320.04 96.52) (xy 314.96 96.52)) (stroke (width 0) (type default)))
+(global_label "H2S_WE_SUM" (shape bidirectional) (at 314.96 96.52 180) (effects (font (size 0.9 0.9)) (justify right)))
+(wire (pts (xy 350.52 96.52) (xy 355.6 96.52)) (stroke (width 0) (type default)))
+(global_label "H2S_WE_OUT" (shape bidirectional) (at 355.6 96.52 0) (effects (font (size 0.9 0.9)) (justify left)))
 )

Commit message: Finalize Skylark signal-chain updates and remove obsolete artifacts
Parts:
- C54: value 1uF -> 10uF; footprint Skylark:Capacitor_SMD__C_0603_1608Metric -> Skylark:Capacitor_SMD__C_0805_2012Metric; MPN GRM188R71E105KA12D -> GRM21BR61A106KE19L
Changed lines of the file:
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@@
 (symbol (lib_id "Groundlark:Part_C54") (at 142.24 38.1 0) (unit 1) (in_bom yes) (on_board yes) (dnp no)
               (property "Reference" "C54" (at 142.24 31.560000000000002 0) (effects (font (size 1.27 1.27))))
-              (property "Value" "1uF" (at 142.24 34.06 0) (effects (font (size 1.0 1.0))))
-              (property "Footprint" "Skylark:Capacitor_SMD__C_0603_1608Metric" (at 142.24 38.1 0) (effects (font (size 1 1)) hide))
-              (property "MPN" "GRM188R71E105KA12D" (at 142.24 38.1 0) (effects (font (size 1 1)) hide))
+              (property "Value" "10uF" (at 142.24 34.06 0) (effects (font (size 1.0 1.0))))
+              (property "Footprint" "Skylark:Capacitor_SMD__C_0805_2012Metric" (at 142.24 38.1 0) (effects (font (size 1 1)) hide))
+              (property "MPN" "GRM21BR61A106KE19L" (at 142.24 38.1 0) (effects (font (size 1 1)) hide))
               (instances (project "skylark-usb" (path "/dafe1df7-5e39-58a9-9d86-b1c10fa6f345/c60510a4-912f-56f4-a510-e17dcca6cdbf" (reference "C54") (unit 1)))))
 (wire (pts (xy 127.0 38.1) (xy 121.92 38.1)) (stroke (width 0) (type default)))
