File: hw/skylark-usb/boards/skylark-usb/06_Environment-page-01.kicad_sch (KiCad schematic)
At the start: 5 parts, among them U11 SHT40-AD1F-R2, U12 BMP390

Commit message: Finalize Skylark signal-chain updates and remove obsolete artifacts
Parts:
- U12: value BMP390 -> BMP388; footprint Skylark:BMP390 -> Skylark:BMP388; MPN BMP390 -> BMP388
Changed lines of the file:
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@@
 (symbol (lib_id "Groundlark:Part_U12") (at 238.76 43.18 0) (unit 1) (in_bom yes) (on_board yes) (dnp no)
               (property "Reference" "U12" (at 238.76 31.560000000000002 0) (effects (font (size 1.27 1.27))))
-              (property "Value" "BMP390" (at 238.76 34.06 0) (effects (font (size 1.0 1.0))))
-              (property "Footprint" "Skylark:BMP390" (at 238.76 43.18 0) (effects (font (size 1 1)) hide))
-              (property "MPN" "BMP390" (at 238.76 43.18 0) (effects (font (size 1 1)) hide))
+              (property "Value" "BMP388" (at 238.76 34.06 0) (effects (font (size 1.0 1.0))))
+              (property "Footprint" "Skylark:BMP388" (at 238.76 43.18 0) (effects (font (size 1 1)) hide))
+              (property "MPN" "BMP388" (at 238.76 43.18 0) (effects (font (size 1 1)) hide))
               (instances (project "skylark-usb" (path "/dafe1df7-5e39-58a9-9d86-b1c10fa6f345/40888c6d-2ce3-5d77-bcb4-504f672fefd3" (reference "U12") (unit 1)))))
 (wire (pts (xy 223.52 38.1) (xy 218.44 38.1)) (stroke (width 0) (type default)))
