File: hw/groundlark-fpga-hat/boards/groundlark-daqhat-01/03-geophone-page-01.kicad_sch (KiCad schematic)
At the start: 12 parts, among them J90 GEO + / - / SHIELD, U22 ADS122C04

Commit message: Use horizontal geophone connector and publish detailed enclosure render
Synchronize J90 routing, native SES, assembly mapping, enclosure fit, models and validation. Add a 4K clear-PETG README render and derive assembly PDF part identities from package procurement. Preserve Git-normalized source bindings and original validation/render input hashes. Generated JLCPCB packages remain local.
Parts:
- J90: footprint Groundlark:Connector_Phoenix_MC__PhoenixContact_MCV_1,5_3-G-3.81_1x03_P3.81mm_Vertical -> Groundlark:Connector_Phoenix_MC__PhoenixContact_MC_1,5_3-G-3.81_1x03_P3.81mm_Horizontal; MPN 1803439 -> 1803280
Changed lines of the file:
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@@
               (property "Reference" "J90" (at 147.32 31.560000000000002 0) (effects (font (size 1.27 1.27))))
               (property "Value" "GEO + / - / SHIELD" (at 147.32 34.06 0) (effects (font (size 1.0 1.0))))
-              (property "Footprint" "Groundlark:Connector_Phoenix_MC__PhoenixContact_MCV_1,5_3-G-3.81_1x03_P3.81mm_Vertical" (at 147.32 39.370000000000005 0) (effects (font (size 1 1)) hide))
-              (property "MPN" "1803439" (at 147.32 39.370000000000005 0) (effects (font (size 1 1)) hide))
+              (property "Footprint" "Groundlark:Connector_Phoenix_MC__PhoenixContact_MC_1,5_3-G-3.81_1x03_P3.81mm_Horizontal" (at 147.32 39.370000000000005 0) (effects (font (size 1 1)) hide))
+              (property "MPN" "1803280" (at 147.32 39.370000000000005 0) (effects (font (size 1 1)) hide))
               (instances (project "groundlark-daqhat-01" (path "/de5c43d7-546f-5b4d-b587-d8dfceb38170/fc4af920-ec4d-5175-b830-5c947dce5acb" (reference "J90") (unit 1)))))
 (wire (pts (xy 132.08 38.1) (xy 127.0 38.1)) (stroke (width 0) (type default)))
