File: hw/groundlark-fpga-hat/boards/groundlark-daqhat-01/01-host-power-page-01.kicad_sch (KiCad schematic)
At the start: 9 parts, among them J1 Raspberry Pi 40-pin, U1 24LC32A

Commit message: Add TI Pi power supervision and expand DAQHAT enclosure
Connections:
- net PI_SHUTDOWN_N: now reaches J1.31
- net PI_HALTED: now reaches J1.33
- no-connect marks 3 -> 1
Changed lines of the file:
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@@
-(kicad_sch (version 20230121) (generator eeschema) (paper "A3") (title_block (title "Groundlark DAQHAT-01 / 01-host-power-page-01") (date "2026-09-24") (rev "DAQHAT-01"))
+(kicad_sch (version 20230121) (generator eeschema) (paper "A3") (title_block (title "Groundlark DAQHAT-01 / 01-host-power-page-01") (date "2026-09-30") (rev "DAQHAT-01"))
 (symbol (lib_id "Groundlark:Part_J1") (at 50.8 62.230000000000004 0) (unit 1) (in_bom yes) (on_board yes) (dnp no)
               (property "Reference" "J1" (at 50.8 31.560000000000002 0) (effects (font (size 1.27 1.27))))
@@
 (wire (pts (xy 66.04 60.96) (xy 71.12 60.96)) (stroke (width 0) (type default)))
 (global_label "GND" (shape bidirectional) (at 71.12 60.96 0) (effects (font (size 0.9 0.9)) (justify left)))
-(no_connect (at 66.04 63.5))
+(wire (pts (xy 66.04 63.5) (xy 71.12 63.5)) (stroke (width 0) (type default)))
+(global_label "PI_SHUTDOWN_N" (shape bidirectional) (at 71.12 63.5 0) (effects (font (size 0.9 0.9)) (justify left)))
 (wire (pts (xy 66.04 66.04) (xy 71.12 66.04)) (stroke (width 0) (type default)))
 (global_label "PI_LINK_DQ3" (shape bidirectional) (at 71.12 66.04 0) (effects (font (size 0.9 0.9)) (justify left)))
-(no_connect (at 66.04 68.58))
+(wire (pts (xy 66.04 68.58) (xy 71.12 68.58)) (stroke (width 0) (type default)))
+(global_label "PI_HALTED" (shape bidirectional) (at 71.12 68.58 0) (effects (font (size 0.9 0.9)) (justify left)))
 (wire (pts (xy 66.04 71.12) (xy 71.12 71.12)) (stroke (width 0) (type default)))
 (global_label "GND" (shape bidirectional) (at 71.12 71.12 0) (effects (font (size 0.9 0.9)) (justify left)))
@@
 (symbol (lib_id "Groundlark:PWR_FLAG") (at 289.56 274.32 0) (unit 1) (in_bom no) (on_board no) (property "Reference" "#FLG06" (at 289.56 274.32 0) (effects (font (size 1 1)) hide)) (property "Value" "PWR_FLAG" (at 289.56 274.32 0) (effects (font (size 1 1)) hide)) (instances (project "groundlark-daqhat-01" (path "/de5c43d7-546f-5b4d-b587-d8dfceb38170/06af75fa-1640-573a-99d0-a877f250c10b" (reference "#FLG06") (unit 1)))))
 (global_label "GEO_AVDD" (shape input) (at 289.56 274.32 0) (effects (font (size 1.0 1.0)) (justify left)))
+(symbol (lib_id "Groundlark:PWR_FLAG") (at 340.35999999999996 274.32 0) (unit 1) (in_bom no) (on_board no) (property "Reference" "#FLG07" (at 340.35999999999996 274.32 0) (effects (font (size 1 1)) hide)) (property "Value" "PWR_FLAG" (at 340.35999999999996 274.32 0) (effects (font (size 1 1)) hide)) (instances (project "groundlark-daqhat-01" (path "/de5c43d7-546f-5b4d-b587-d8dfceb38170/06af75fa-1640-573a-99d0-a877f250c10b" (reference "#FLG07") (unit 1)))))
+(global_label "SUP_3V3" (shape input) (at 340.35999999999996 274.32 0) (effects (font (size 1.0 1.0)) (justify left)))
 )

Commit message: Add Groundlark GNSS timing, SMA access and calibration workflow
Connections:
- net GNSS_PPS: now reaches J1.18
- no-connect marks 1 -> 0
Changed lines of the file:
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@@
 (wire (pts (xy 35.56 78.74) (xy 30.48 78.74)) (stroke (width 0) (type default)))
 (global_label "PI_3V3" (shape bidirectional) (at 30.48 78.74 180) (effects (font (size 0.9 0.9)) (justify right)))
-(no_connect (at 35.56 81.28))
+(wire (pts (xy 35.56 81.28) (xy 30.48 81.28)) (stroke (width 0) (type default)))
+(global_label "GNSS_PPS" (shape bidirectional) (at 30.48 81.28 180) (effects (font (size 0.9 0.9)) (justify right)))
 (wire (pts (xy 35.56 83.82) (xy 30.48 83.82)) (stroke (width 0) (type default)))
 (global_label "PI_SPI_MOSI" (shape bidirectional) (at 30.48 83.82 180) (effects (font (size 0.9 0.9)) (justify right)))
