File: hw/groundlark-fpga-hat/boards/groundlark-daqhat-01/04-gnss-page-01.kicad_sch (KiCad schematic)
At the start: 10 parts, among them J140 GNSS ANT / 3V3, U140 TPS70933, U21 MAX-M10S-00B

Commit message: Fix Groundlark power and GNSS electrical faults
Parts:
- added C151: 10n, Groundlark:SUP_C_0603_1608Metric, symbol Groundlark:Part_C151
- added U141: TPS2553, Groundlark:GNSS_SOT23_6, symbol Groundlark:Part_U141
- C146, C149, C150: MPN GRM21BR71A475KA73L -> GRM21BR71C475KA73L
Connections:
- net GND: now also C151.2, U141.2
- net GNSS_BIAS: now also C151.1, U141.6; no longer C150.1, U140.5
- new net GNSS_LDO: C150.1, U140.5, U141.1, U141.3, U141.5
- no-connect marks 10 -> 11
Changed lines of the file:
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@@
               (property "Value" "4.7u" (at 243.83999999999997 34.06 0) (effects (font (size 1.0 1.0))))
               (property "Footprint" "Groundlark:Capacitor_SMD__C_0805_2012Metric" (at 243.83999999999997 38.1 0) (effects (font (size 1 1)) hide))
-              (property "MPN" "GRM21BR71A475KA73L" (at 243.83999999999997 38.1 0) (effects (font (size 1 1)) hide))
+              (property "MPN" "GRM21BR71C475KA73L" (at 243.83999999999997 38.1 0) (effects (font (size 1 1)) hide))
               (instances (project "groundlark-daqhat-01" (path "/de5c43d7-546f-5b4d-b587-d8dfceb38170/63456fc1-bcd1-564c-918b-1145ac1e9ff5" (reference "C146") (unit 1)))))
 (wire (pts (xy 228.6 38.1) (xy 223.52 38.1)) (stroke (width 0) (type default)))
@@
 (no_connect (at 259.08 86.36))
 (wire (pts (xy 259.08 88.9) (xy 264.16 88.9)) (stroke (width 0) (type default)))
-(global_label "GNSS_BIAS" (shape bidirectional) (at 264.16 88.9 0) (effects (font (size 0.9 0.9)) (justify left)))
+(global_label "GNSS_LDO" (shape bidirectional) (at 264.16 88.9 0) (effects (font (size 0.9 0.9)) (justify left)))
 (symbol (lib_id "Groundlark:Part_C149") (at 340.35999999999996 86.36 0) (unit 1) (in_bom yes) (on_board yes) (dnp no)
               (property "Reference" "C149" (at 340.35999999999996 79.82 0) (effects (font (size 1.27 1.27))))
               (property "Value" "4.7u" (at 340.35999999999996 82.32 0) (effects (font (size 1.0 1.0))))
               (property "Footprint" "Groundlark:Capacitor_SMD__C_0805_2012Metric" (at 340.35999999999996 86.36 0) (effects (font (size 1 1)) hide))
-              (property "MPN" "GRM21BR71A475KA73L" (at 340.35999999999996 86.36 0) (effects (font (size 1 1)) hide))
+              (property "MPN" "GRM21BR71C475KA73L" (at 340.35999999999996 86.36 0) (effects (font (size 1 1)) hide))
               (instances (project "groundlark-daqhat-01" (path "/de5c43d7-546f-5b4d-b587-d8dfceb38170/63456fc1-bcd1-564c-918b-1145ac1e9ff5" (reference "C149") (unit 1)))))
 (wire (pts (xy 325.12 86.36) (xy 320.04 86.36)) (stroke (width 0) (type default)))
@@
               (property "Value" "4.7u" (at 50.8 115.33999999999999 0) (effects (font (size 1.0 1.0))))
               (property "Footprint" "Groundlark:Capacitor_SMD__C_0805_2012Metric" (at 50.8 119.38 0) (effects (font (size 1 1)) hide))
-              (property "MPN" "GRM21BR71A475KA73L" (at 50.8 119.38 0) (effects (font (size 1 1)) hide))
+              (property "MPN" "GRM21BR71C475KA73L" (at 50.8 119.38 0) (effects (font (size 1 1)) hide))
               (instances (project "groundlark-daqhat-01" (path "/de5c43d7-546f-5b4d-b587-d8dfceb38170/63456fc1-bcd1-564c-918b-1145ac1e9ff5" (reference "C150") (unit 1)))))
 (wire (pts (xy 35.56 119.38) (xy 30.48 119.38)) (stroke (width 0) (type default)))
-(global_label "GNSS_BIAS" (shape bidirectional) (at 30.48 119.38 180) (effects (font (size 0.9 0.9)) (justify right)))
+(global_label "GNSS_LDO" (shape bidirectional) (at 30.48 119.38 180) (effects (font (size 0.9 0.9)) (justify right)))
 (wire (pts (xy 66.04 119.38) (xy 71.12 119.38)) (stroke (width 0) (type default)))
 (global_label "GND" (shape bidirectional) (at 71.12 119.38 0) (effects (font (size 0.9 0.9)) (justify left)))
@@
 (wire (pts (xy 162.56 119.38) (xy 167.64 119.38)) (stroke (width 0) (type default)))
 (global_label "GND" (shape bidirectional) (at 167.64 119.38 0) (effects (font (size 0.9 0.9)) (justify left)))
+(symbol (lib_id "Groundlark:Part_U141") (at 243.83999999999997 121.91999999999999 0) (unit 1) (in_bom yes) (on_board yes) (dnp no)
+              (property "Reference" "U141" (at 243.83999999999997 112.83999999999999 0) (effects (font (size 1.27 1.27))))
+              (property "Value" "TPS2553" (at 243.83999999999997 115.33999999999999 0) (effects (font (size 1.0 1.0))))
+              (property "Footprint" "Groundlark:GNSS_SOT23_6" (at 243.83999999999997 121.91999999999999 0) (effects (font (size 1 1)) hide))
+              (property "MPN" "TPS2553DBVR" (at 243.83999999999997 121.91999999999999 0) (effects (font (size 1 1)) hide))
+              (instances (project "groundlark-daqhat-01" (path "/de5c43d7-546f-5b4d-b587-d8dfceb38170/63456fc1-bcd1-564c-918b-1145ac1e9ff5" (reference "U141") (unit 1)))))
+(wire (pts (xy 228.6 119.38) (xy 223.52 119.38)) (stroke (width 0) (type default)))
+(global_label "GNSS_LDO" (shape bidirectional) (at 223.52 119.38 180) (effects (font (size 0.9 0.9)) (justify right)))
+(wire (pts (xy 228.6 121.92) (xy 223.52 121.92)) (stroke (width 0) (type default)))
+(global_label "GND" (shape bidirectional) (at 223.52 121.92 180) (effects (font (size 0.9 0.9)) (justify right)))
+(wire (pts (xy 228.6 124.46) (xy 223.52 124.46)) (stroke (width 0) (type default)))
+(global_label "GNSS_LDO" (shape bidirectional) (at 223.52 124.46 180) (effects (font (size 0.9 0.9)) (justify right)))
+(no_connect (at 259.08 119.38))
+(wire (pts (xy 259.08 121.92) (xy 264.16 121.92)) (stroke (width 0) (type default)))
+(global_label "GNSS_LDO" (shape bidirectional) (at 264.16 121.92 0) (effects (font (size 0.9 0.9)) (justify left)))
+(wire (pts (xy 259.08 124.46) (xy 264.16 124.46)) (stroke (width 0) (type default)))
+(global_label "GNSS_BIAS" (shape bidirectional) (at 264.16 124.46 0) (effects (font (size 0.9 0.9)) (justify left)))
+(symbol (lib_id "Groundlark:Part_C151") (at 340.35999999999996 119.38 0) (unit 1) (in_bom yes) (on_board yes) (dnp no)
+              (property "Reference" "C151" (at 340.35999999999996 112.83999999999999 0) (effects (font (size 1.27 1.27))))
+              (property "Value" "10n" (at 340.35999999999996 115.33999999999999 0) (effects (font (size 1.0 1.0))))
+              (property "Footprint" "Groundlark:SUP_C_0603_1608Metric" (at 340.35999999999996 119.38 0) (effects (font (size 1 1)) hide))
+              (property "MPN" "GRM188R71H103KA01D" (at 340.35999999999996 119.38 0) (effects (font (size 1 1)) hide))
+              (instances (project "groundlark-daqhat-01" (path "/de5c43d7-546f-5b4d-b587-d8dfceb38170/63456fc1-bcd1-564c-918b-1145ac1e9ff5" (reference "C151") (unit 1)))))
+(wire (pts (xy 325.12 119.38) (xy 320.04 119.38)) (stroke (width 0) (type default)))
+(global_label "GNSS_BIAS" (shape bidirectional) (at 320.04 119.38 180) (effects (font (size 0.9 0.9)) (justify right)))
+(wire (pts (xy 355.6 119.38) (xy 360.68 119.38)) (stroke (width 0) (type default)))
+(global_label "GND" (shape bidirectional) (at 360.68 119.38 0) (effects (font (size 0.9 0.9)) (justify left)))
 )
