File: hw/groundlark-fpga-hat/boards/groundlark-daqhat-01/06-supply-isolation-page-02.kicad_sch (KiCad schematic)
At the start: 9 parts, among them U43 ISO1640BDR

Commit message: Fix Groundlark power and GNSS electrical faults
Connections:
- net I2C_SCL: now also U43.3 (SCL1); no longer U43.6 (SCL2)
- net I2C_SDA: now also U43.2 (SDA1); no longer U43.7 (SDA2)
- net PI_3V3: now also C49.1, U43.8 (VCC2); no longer C48.1, U43.1 (VCC1)
- net PI_I2C_SCL: now also U43.6 (SCL2); no longer U43.3 (SCL1)
- net PI_I2C_SDA: now also U43.7 (SDA2); no longer U43.2 (SDA1)
- net SENS_3V3: now also C48.1, U43.1 (VCC1); no longer C49.1, U43.8 (VCC2)
Changed lines of the file:
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@@
               (instances (project "groundlark-daqhat-01" (path "/de5c43d7-546f-5b4d-b587-d8dfceb38170/f56ecc3e-4553-5db6-a260-32f4de25afe3" (reference "U43") (unit 1)))))
 (wire (pts (xy 132.08 38.1) (xy 127.0 38.1)) (stroke (width 0) (type default)))
-(global_label "PI_3V3" (shape bidirectional) (at 127.0 38.1 180) (effects (font (size 0.9 0.9)) (justify right)))
+(global_label "SENS_3V3" (shape bidirectional) (at 127.0 38.1 180) (effects (font (size 0.9 0.9)) (justify right)))
 (wire (pts (xy 132.08 40.64) (xy 127.0 40.64)) (stroke (width 0) (type default)))
-(global_label "PI_I2C_SDA" (shape bidirectional) (at 127.0 40.64 180) (effects (font (size 0.9 0.9)) (justify right)))
+(global_label "I2C_SDA" (shape bidirectional) (at 127.0 40.64 180) (effects (font (size 0.9 0.9)) (justify right)))
 (wire (pts (xy 132.08 43.18) (xy 127.0 43.18)) (stroke (width 0) (type default)))
-(global_label "PI_I2C_SCL" (shape bidirectional) (at 127.0 43.18 180) (effects (font (size 0.9 0.9)) (justify right)))
+(global_label "I2C_SCL" (shape bidirectional) (at 127.0 43.18 180) (effects (font (size 0.9 0.9)) (justify right)))
 (wire (pts (xy 132.08 45.72) (xy 127.0 45.72)) (stroke (width 0) (type default)))
 (global_label "GND" (shape bidirectional) (at 127.0 45.72 180) (effects (font (size 0.9 0.9)) (justify right)))
@@
 (global_label "GND" (shape bidirectional) (at 167.64 38.1 0) (effects (font (size 0.9 0.9)) (justify left)))
 (wire (pts (xy 162.56 40.64) (xy 167.64 40.64)) (stroke (width 0) (type default)))
-(global_label "I2C_SCL" (shape bidirectional) (at 167.64 40.64 0) (effects (font (size 0.9 0.9)) (justify left)))
+(global_label "PI_I2C_SCL" (shape bidirectional) (at 167.64 40.64 0) (effects (font (size 0.9 0.9)) (justify left)))
 (wire (pts (xy 162.56 43.18) (xy 167.64 43.18)) (stroke (width 0) (type default)))
-(global_label "I2C_SDA" (shape bidirectional) (at 167.64 43.18 0) (effects (font (size 0.9 0.9)) (justify left)))
+(global_label "PI_I2C_SDA" (shape bidirectional) (at 167.64 43.18 0) (effects (font (size 0.9 0.9)) (justify left)))
 (wire (pts (xy 162.56 45.72) (xy 167.64 45.72)) (stroke (width 0) (type default)))
-(global_label "SENS_3V3" (shape bidirectional) (at 167.64 45.72 0) (effects (font (size 0.9 0.9)) (justify left)))
+(global_label "PI_3V3" (shape bidirectional) (at 167.64 45.72 0) (effects (font (size 0.9 0.9)) (justify left)))
 (symbol (lib_id "Groundlark:Part_C48") (at 243.83999999999997 38.1 0) (unit 1) (in_bom yes) (on_board yes) (dnp no)
               (property "Reference" "C48" (at 243.83999999999997 31.560000000000002 0) (effects (font (size 1.27 1.27))))
@@
               (instances (project "groundlark-daqhat-01" (path "/de5c43d7-546f-5b4d-b587-d8dfceb38170/f56ecc3e-4553-5db6-a260-32f4de25afe3" (reference "C48") (unit 1)))))
 (wire (pts (xy 228.6 38.1) (xy 223.52 38.1)) (stroke (width 0) (type default)))
-(global_label "PI_3V3" (shape bidirectional) (at 223.52 38.1 180) (effects (font (size 0.9 0.9)) (justify right)))
+(global_label "SENS_3V3" (shape bidirectional) (at 223.52 38.1 180) (effects (font (size 0.9 0.9)) (justify right)))
 (wire (pts (xy 259.08 38.1) (xy 264.16 38.1)) (stroke (width 0) (type default)))
 (global_label "GND" (shape bidirectional) (at 264.16 38.1 0) (effects (font (size 0.9 0.9)) (justify left)))
@@
               (instances (project "groundlark-daqhat-01" (path "/de5c43d7-546f-5b4d-b587-d8dfceb38170/f56ecc3e-4553-5db6-a260-32f4de25afe3" (reference "C49") (unit 1)))))
 (wire (pts (xy 325.12 38.1) (xy 320.04 38.1)) (stroke (width 0) (type default)))
-(global_label "SENS_3V3" (shape bidirectional) (at 320.04 38.1 180) (effects (font (size 0.9 0.9)) (justify right)))
+(global_label "PI_3V3" (shape bidirectional) (at 320.04 38.1 180) (effects (font (size 0.9 0.9)) (justify right)))
 (wire (pts (xy 355.6 38.1) (xy 360.68 38.1)) (stroke (width 0) (type default)))
 (global_label "GND" (shape bidirectional) (at 360.68 38.1 0) (effects (font (size 0.9 0.9)) (justify left)))
