File: hw/groundlark-fpga-hat/boards/groundlark-daqhat-01/09-fpga-power-page-01.kicad_sch (KiCad schematic)
At the start: 6 parts

Commit message: Add TI Pi power supervision and expand DAQHAT enclosure
Parts:
- added D80: B340A, Groundlark:PWR_D_SMA, symbol Groundlark:Part_D80
- added D81: SMAJ15A, Groundlark:PWR_D_SMA, symbol Groundlark:Part_D81
- added F80: 2A fast, Groundlark:PWR_Fuse_1206_3216Metric, symbol Groundlark:Part_F80
- added J83: 12V DC / CENTER +, Groundlark:PWR_BarrelJack_CUI_PJ-102AH_Horizontal, symbol Groundlark:Part_J83
- added R120: 10k, Groundlark:PWR_R_0603_1608Metric, symbol Groundlark:Part_R120
- added U80: TPSM53603, Groundlark:PWR_Texas_B3QFN-14-1EP_5x5.5mm_P0.65mm, symbol Groundlark:Part_U80
Connections:
- net FPGA_VIN: now also R120.1, U80.7 (VOUT), U80.8 (VOUT)
- net GND: now also D81.2 (A), J83.2 (SLEEVE), U80.10 (NC_GND), U80.11 (NC_GND), U80.12 (AGND), U80.15 (PGND), U80.3 (NC_GND)
- new net BUCK_EN: U80.2 (EN)
- new net BUCK_FB: R120.2, U80.9 (FB)
- new net EXT_12V: F80.1, J83.1 (CENTER)
- new net FPGA_EN1: U80.6 (PGOOD)
- new net FUSED_12V: D80.2 (A), F80.2
- new net PROTECTED_12V: D80.1 (K), D81.1 (K), U80.1 (VIN), U80.14 (VIN)
- no-connect marks 0 -> 4
Changed lines of the file:
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@@
-(kicad_sch (version 20230121) (generator eeschema) (paper "A3") (title_block (title "Groundlark DAQHAT-01 / 09-fpga-power-page-01") (date "2026-09-24") (rev "DAQHAT-01"))
+(kicad_sch (version 20230121) (generator eeschema) (paper "A3") (title_block (title "Groundlark DAQHAT-01 / 09-fpga-power-page-01") (date "2026-09-30") (rev "DAQHAT-01"))
 (symbol (lib_id "Groundlark:Part_C80") (at 50.8 38.1 0) (unit 1) (in_bom yes) (on_board yes) (dnp no)
               (property "Reference" "C80" (at 50.8 31.560000000000002 0) (effects (font (size 1.27 1.27))))
@@
 (wire (pts (xy 162.56 66.04) (xy 167.64 66.04)) (stroke (width 0) (type default)))
 (global_label "GND" (shape bidirectional) (at 167.64 66.04 0) (effects (font (size 0.9 0.9)) (justify left)))
+(symbol (lib_id "Groundlark:Part_J83") (at 243.83999999999997 67.31 0) (unit 1) (in_bom yes) (on_board yes) (dnp no)
+              (property "Reference" "J83" (at 243.83999999999997 59.5 0) (effects (font (size 1.27 1.27))))
+              (property "Value" "12V DC / CENTER +" (at 243.83999999999997 62.0 0) (effects (font (size 1.0 1.0))))
+              (property "Footprint" "Groundlark:PWR_BarrelJack_CUI_PJ-102AH_Horizontal" (at 243.83999999999997 67.31 0) (effects (font (size 1 1)) hide))
+              (property "MPN" "PJ-102AH" (at 243.83999999999997 67.31 0) (effects (font (size 1 1)) hide))
+              (instances (project "groundlark-daqhat-01" (path "/de5c43d7-546f-5b4d-b587-d8dfceb38170/4268834e-07e4-571f-acec-28e289faab28" (reference "J83") (unit 1)))))
+(wire (pts (xy 228.6 66.04) (xy 223.52 66.04)) (stroke (width 0) (type default)))
+(global_label "EXT_12V" (shape bidirectional) (at 223.52 66.04 180) (effects (font (size 0.9 0.9)) (justify right)))
+(wire (pts (xy 228.6 68.58) (xy 223.52 68.58)) (stroke (width 0) (type default)))
+(global_label "GND" (shape bidirectional) (at 223.52 68.58 180) (effects (font (size 0.9 0.9)) (justify right)))
+(no_connect (at 259.08 66.04))
+(symbol (lib_id "Groundlark:Part_F80") (at 340.35999999999996 66.04 0) (unit 1) (in_bom yes) (on_board yes) (dnp no)
+              (property "Reference" "F80" (at 340.35999999999996 59.5 0) (effects (font (size 1.27 1.27))))
+              (property "Value" "2A fast" (at 340.35999999999996 62.0 0) (effects (font (size 1.0 1.0))))
+              (property "Footprint" "Groundlark:PWR_Fuse_1206_3216Metric" (at 340.35999999999996 66.04 0) (effects (font (size 1 1)) hide))
+              (property "MPN" "0467002.NR" (at 340.35999999999996 66.04 0) (effects (font (size 1 1)) hide))
+              (instances (project "groundlark-daqhat-01" (path "/de5c43d7-546f-5b4d-b587-d8dfceb38170/4268834e-07e4-571f-acec-28e289faab28" (reference "F80") (unit 1)))))
+(wire (pts (xy 325.12 66.04) (xy 320.04 66.04)) (stroke (width 0) (type default)))
+(global_label "EXT_12V" (shape bidirectional) (at 320.04 66.04 180) (effects (font (size 0.9 0.9)) (justify right)))
+(wire (pts (xy 355.6 66.04) (xy 360.68 66.04)) (stroke (width 0) (type default)))
+(global_label "FUSED_12V" (shape bidirectional) (at 360.68 66.04 0) (effects (font (size 0.9 0.9)) (justify left)))
+(symbol (lib_id "Groundlark:Part_D80") (at 50.8 96.52000000000001 0) (unit 1) (in_bom yes) (on_board yes) (dnp no)
+              (property "Reference" "D80" (at 50.8 89.98 0) (effects (font (size 1.27 1.27))))
+              (property "Value" "B340A" (at 50.8 92.48 0) (effects (font (size 1.0 1.0))))
+              (property "Footprint" "Groundlark:PWR_D_SMA" (at 50.8 96.52000000000001 0) (effects (font (size 1 1)) hide))
+              (property "MPN" "B340A-13-F" (at 50.8 96.52000000000001 0) (effects (font (size 1 1)) hide))
+              (instances (project "groundlark-daqhat-01" (path "/de5c43d7-546f-5b4d-b587-d8dfceb38170/4268834e-07e4-571f-acec-28e289faab28" (reference "D80") (unit 1)))))
+(wire (pts (xy 35.56 96.52) (xy 30.48 96.52)) (stroke (width 0) (type default)))
+(global_label "PROTECTED_12V" (shape bidirectional) (at 30.48 96.52 180) (effects (font (size 0.9 0.9)) (justify right)))
+(wire (pts (xy 66.04 96.52) (xy 71.12 96.52)) (stroke (width 0) (type default)))
+(global_label "FUSED_12V" (shape bidirectional) (at 71.12 96.52 0) (effects (font (size 0.9 0.9)) (justify left)))
+(symbol (lib_id "Groundlark:Part_D81") (at 147.32 96.52000000000001 0) (unit 1) (in_bom yes) (on_board yes) (dnp no)
+              (property "Reference" "D81" (at 147.32 89.98 0) (effects (font (size 1.27 1.27))))
+              (property "Value" "SMAJ15A" (at 147.32 92.48 0) (effects (font (size 1.0 1.0))))
+              (property "Footprint" "Groundlark:PWR_D_SMA" (at 147.32 96.52000000000001 0) (effects (font (size 1 1)) hide))
+              (property "MPN" "SMAJ15A-13-F" (at 147.32 96.52000000000001 0) (effects (font (size 1 1)) hide))
+              (instances (project "groundlark-daqhat-01" (path "/de5c43d7-546f-5b4d-b587-d8dfceb38170/4268834e-07e4-571f-acec-28e289faab28" (reference "D81") (unit 1)))))
+(wire (pts (xy 132.08 96.52) (xy 127.0 96.52)) (stroke (width 0) (type default)))
+(global_label "PROTECTED_12V" (shape bidirectional) (at 127.0 96.52 180) (effects (font (size 0.9 0.9)) (justify right)))
+(wire (pts (xy 162.56 96.52) (xy 167.64 96.52)) (stroke (width 0) (type default)))
+(global_label "GND" (shape bidirectional) (at 167.64 96.52 0) (effects (font (size 0.9 0.9)) (justify left)))
+(symbol (lib_id "Groundlark:Part_U80") (at 243.83999999999997 105.41 0) (unit 1) (in_bom yes) (on_board yes) (dnp no)
+              (property "Reference" "U80" (at 243.83999999999997 89.98 0) (effects (font (size 1.27 1.27))))
+              (property "Value" "TPSM53603" (at 243.83999999999997 92.48 0) (effects (font (size 1.0 1.0))))
+              (property "Footprint" "Groundlark:PWR_Texas_B3QFN-14-1EP_5x5.5mm_P0.65mm" (at 243.83999999999997 105.41 0) (effects (font (size 1 1)) hide))
+              (property "MPN" "TPSM53603RDAR" (at 243.83999999999997 105.41 0) (effects (font (size 1 1)) hide))
+              (instances (project "groundlark-daqhat-01" (path "/de5c43d7-546f-5b4d-b587-d8dfceb38170/4268834e-07e4-571f-acec-28e289faab28" (reference "U80") (unit 1)))))
+(wire (pts (xy 228.6 96.52) (xy 223.52 96.52)) (stroke (width 0) (type default)))
+(global_label "PROTECTED_12V" (shape bidirectional) (at 223.52 96.52 180) (effects (font (size 0.9 0.9)) (justify right)))
+(wire (pts (xy 228.6 99.06) (xy 223.52 99.06)) (stroke (width 0) (type default)))
+(global_label "BUCK_EN" (shape bidirectional) (at 223.52 99.06 180) (effects (font (size 0.9 0.9)) (justify right)))
+(wire (pts (xy 228.6 101.6) (xy 223.52 101.6)) (stroke (width 0) (type default)))
+(global_label "GND" (shape bidirectional) (at 223.52 101.6 180) (effects (font (size 0.9 0.9)) (justify right)))
+(no_connect (at 228.6 104.14))
+(no_connect (at 228.6 106.68))
+(wire (pts (xy 228.6 109.22) (xy 223.52 109.22)) (stroke (width 0) (type default)))
+(global_label "FPGA_EN1" (shape bidirectional) (at 223.52 109.22 180) (effects (font (size 0.9 0.9)) (justify right)))
+(wire (pts (xy 228.6 111.76) (xy 223.52 111.76)) (stroke (width 0) (type default)))
+(global_label "FPGA_VIN" (shape bidirectional) (at 223.52 111.76 180) (effects (font (size 0.9 0.9)) (justify right)))
+(wire (pts (xy 228.6 114.3) (xy 223.52 114.3)) (stroke (width 0) (type default)))
+(global_label "FPGA_VIN" (shape bidirectional) (at 223.52 114.3 180) (effects (font (size 0.9 0.9)) (justify right)))
+(wire (pts (xy 259.08 96.52) (xy 264.16 96.52)) (stroke (width 0) (type default)))
+(global_label "BUCK_FB" (shape bidirectional) (at 264.16 96.52 0) (effects (font (size 0.9 0.9)) (justify left)))
+(wire (pts (xy 259.08 99.06) (xy 264.16 99.06)) (stroke (width 0) (type default)))
+(global_label "GND" (shape bidirectional) (at 264.16 99.06 0) (effects (font (size 0.9 0.9)) (justify left)))
+(wire (pts (xy 259.08 101.6) (xy 264.16 101.6)) (stroke (width 0) (type default)))
+(global_label "GND" (shape bidirectional) (at 264.16 101.6 0) (effects (font (size 0.9 0.9)) (justify left)))
+(wire (pts (xy 259.08 104.14) (xy 264.16 104.14)) (stroke (width 0) (type default)))
+(global_label "GND" (shape bidirectional) (at 264.16 104.14 0) (effects (font (size 0.9 0.9)) (justify left)))
+(no_connect (at 259.08 106.68))
+(wire (pts (xy 259.08 109.22) (xy 264.16 109.22)) (stroke (width 0) (type default)))
+(global_label "PROTECTED_12V" (shape bidirectional) (at 264.16 109.22 0) (effects (font (size 0.9 0.9)) (justify left)))
+(wire (pts (xy 259.08 111.76) (xy 264.16 111.76)) (stroke (width 0) (type default)))
+(global_label "GND" (shape bidirectional) (at 264.16 111.76 0) (effects (font (size 0.9 0.9)) (justify left)))
+(symbol (lib_id "Groundlark:Part_R120") (at 340.35999999999996 96.52000000000001 0) (unit 1) (in_bom yes) (on_board yes) (dnp no)
+              (property "Reference" "R120" (at 340.35999999999996 89.98 0) (effects (font (size 1.27 1.27))))
+              (property "Value" "10k" (at 340.35999999999996 92.48 0) (effects (font (size 1.0 1.0))))
+              (property "Footprint" "Groundlark:PWR_R_0603_1608Metric" (at 340.35999999999996 96.52000000000001 0) (effects (font (size 1 1)) hide))
+              (property "MPN" "RT0603BRD0710KL" (at 340.35999999999996 96.52000000000001 0) (effects (font (size 1 1)) hide))
+              (instances (project "groundlark-daqhat-01" (path "/de5c43d7-546f-5b4d-b587-d8dfceb38170/4268834e-07e4-571f-acec-28e289faab28" (reference "R120") (unit 1)))))
+(wire (pts (xy 325.12 96.52) (xy 320.04 96.52)) (stroke (width 0) (type default)))
+(global_label "FPGA_VIN" (shape bidirectional) (at 320.04 96.52 180) (effects (font (size 0.9 0.9)) (justify right)))
+(wire (pts (xy 355.6 96.52) (xy 360.68 96.52)) (stroke (width 0) (type default)))
+(global_label "BUCK_FB" (shape bidirectional) (at 360.68 96.52 0) (effects (font (size 0.9 0.9)) (justify left)))
 )

Commit message: Fix Groundlark power and GNSS electrical faults
Parts:
- F80: value 2A fast -> 0466002.NRHF; MPN 0467002.NR -> 0466002.NRHF
Changed lines of the file:
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@@
 (symbol (lib_id "Groundlark:Part_F80") (at 340.35999999999996 66.04 0) (unit 1) (in_bom yes) (on_board yes) (dnp no)
               (property "Reference" "F80" (at 340.35999999999996 59.5 0) (effects (font (size 1.27 1.27))))
-              (property "Value" "2A fast" (at 340.35999999999996 62.0 0) (effects (font (size 1.0 1.0))))
+              (property "Value" "0466002.NRHF" (at 340.35999999999996 62.0 0) (effects (font (size 1.0 1.0))))
               (property "Footprint" "Groundlark:PWR_Fuse_1206_3216Metric" (at 340.35999999999996 66.04 0) (effects (font (size 1 1)) hide))
-              (property "MPN" "0467002.NR" (at 340.35999999999996 66.04 0) (effects (font (size 1 1)) hide))
+              (property "MPN" "0466002.NRHF" (at 340.35999999999996 66.04 0) (effects (font (size 1 1)) hide))
               (instances (project "groundlark-daqhat-01" (path "/de5c43d7-546f-5b4d-b587-d8dfceb38170/4268834e-07e4-571f-acec-28e289faab28" (reference "F80") (unit 1)))))
 (wire (pts (xy 325.12 66.04) (xy 320.04 66.04)) (stroke (width 0) (type default)))
