File: hw/groundlark-fpga-hat/boards/groundlark-daqhat-01/11-pi-supervisor-page-01.kicad_sch (KiCad schematic)
At the start: 12 parts, among them J130 PI BATTERY 8-18V, U131 TPS70933, U132 TPSM53603

Commit message: Fix Groundlark power and GNSS electrical faults
Parts:
- C130: MPN GRM21BR71A475KA73L -> GRM21BR71C475KA73L
- F130: value 4A fast -> 4A fuse; MPN 0467004.NR -> 0466004.NRHF
Changed lines of the file:
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@@
 (symbol (lib_id "Groundlark:Part_F130") (at 147.32 38.1 0) (unit 1) (in_bom yes) (on_board yes) (dnp no)
               (property "Reference" "F130" (at 147.32 31.560000000000002 0) (effects (font (size 1.27 1.27))))
-              (property "Value" "4A fast" (at 147.32 34.06 0) (effects (font (size 1.0 1.0))))
+              (property "Value" "4A fuse" (at 147.32 34.06 0) (effects (font (size 1.0 1.0))))
               (property "Footprint" "Groundlark:SUP_Fuse_1206_3216Metric" (at 147.32 38.1 0) (effects (font (size 1 1)) hide))
-              (property "MPN" "0467004.NR" (at 147.32 38.1 0) (effects (font (size 1 1)) hide))
+              (property "MPN" "0466004.NRHF" (at 147.32 38.1 0) (effects (font (size 1 1)) hide))
               (instances (project "groundlark-daqhat-01" (path "/de5c43d7-546f-5b4d-b587-d8dfceb38170/42a1d027-f5bb-53a3-b4c0-117ee8ab0995" (reference "F130") (unit 1)))))
 (wire (pts (xy 132.08 38.1) (xy 127.0 38.1)) (stroke (width 0) (type default)))
@@
               (property "Value" "4.7u" (at 147.32 62.0 0) (effects (font (size 1.0 1.0))))
               (property "Footprint" "Groundlark:SUP_C_0805_2012Metric" (at 147.32 66.04 0) (effects (font (size 1 1)) hide))
-              (property "MPN" "GRM21BR71A475KA73L" (at 147.32 66.04 0) (effects (font (size 1 1)) hide))
+              (property "MPN" "GRM21BR71C475KA73L" (at 147.32 66.04 0) (effects (font (size 1 1)) hide))
               (instances (project "groundlark-daqhat-01" (path "/de5c43d7-546f-5b4d-b587-d8dfceb38170/42a1d027-f5bb-53a3-b4c0-117ee8ab0995" (reference "C130") (unit 1)))))
 (wire (pts (xy 132.08 66.04) (xy 127.0 66.04)) (stroke (width 0) (type default)))
