File: hw/groundlark-fpga-hat/boards/groundlark-daqhat-01/11-pi-supervisor-page-02.kicad_sch (KiCad schematic)
At the start: 12 parts, among them U130 MSPM0L1105, U133 TPS22953

Commit message: Fix Groundlark power and GNSS electrical faults
Parts:
- R131: value 2.41k -> 2.43k; MPN RT0603BRD072K41L -> RT0603BRD072K43L
- U130: value MSPM0L1105 -> MSPM0L1106; MPN MSPM0L1105TRHBR -> MSPM0L1106TRHBR
Connections:
- net GND: now also U133.7 (PG_NC)
- no-connect marks 23 -> 22
Changed lines of the file:
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@@
 (symbol (lib_id "Groundlark:Part_R131") (at 50.8 66.04 0) (unit 1) (in_bom yes) (on_board yes) (dnp no)
               (property "Reference" "R131" (at 50.8 59.5 0) (effects (font (size 1.27 1.27))))
-              (property "Value" "2.41k" (at 50.8 62.0 0) (effects (font (size 1.0 1.0))))
+              (property "Value" "2.43k" (at 50.8 62.0 0) (effects (font (size 1.0 1.0))))
               (property "Footprint" "Groundlark:SUP_R_0603_1608Metric" (at 50.8 66.04 0) (effects (font (size 1 1)) hide))
-              (property "MPN" "RT0603BRD072K41L" (at 50.8 66.04 0) (effects (font (size 1 1)) hide))
+              (property "MPN" "RT0603BRD072K43L" (at 50.8 66.04 0) (effects (font (size 1 1)) hide))
               (instances (project "groundlark-daqhat-01" (path "/de5c43d7-546f-5b4d-b587-d8dfceb38170/f6bfc69a-2b11-5d7b-82d1-e99b72f3d077" (reference "R131") (unit 1)))))
 (wire (pts (xy 35.56 66.04) (xy 30.48 66.04)) (stroke (width 0) (type default)))
@@
 (wire (pts (xy 228.6 78.74) (xy 223.52 78.74)) (stroke (width 0) (type default)))
 (global_label "PI_SWITCH_CT" (shape bidirectional) (at 223.52 78.74 180) (effects (font (size 0.9 0.9)) (justify right)))
-(no_connect (at 259.08 66.04))
+(wire (pts (xy 259.08 66.04) (xy 264.16 66.04)) (stroke (width 0) (type default)))
+(global_label "GND" (shape bidirectional) (at 264.16 66.04 0) (effects (font (size 0.9 0.9)) (justify left)))
 (wire (pts (xy 259.08 68.58) (xy 264.16 68.58)) (stroke (width 0) (type default)))
 (global_label "PI_RAW_5V" (shape bidirectional) (at 264.16 68.58 0) (effects (font (size 0.9 0.9)) (justify left)))
@@
 (symbol (lib_id "Groundlark:Part_U130") (at 243.83999999999997 127.0 0) (unit 1) (in_bom yes) (on_board yes) (dnp no)
               (property "Reference" "U130" (at 243.83999999999997 100.14 0) (effects (font (size 1.27 1.27))))
-              (property "Value" "MSPM0L1105" (at 243.83999999999997 102.64 0) (effects (font (size 1.0 1.0))))
+              (property "Value" "MSPM0L1106" (at 243.83999999999997 102.64 0) (effects (font (size 1.0 1.0))))
               (property "Footprint" "Groundlark:SUP_QFN-32-1EP_5x5mm_P0.5mm_EP3.45x3.45mm" (at 243.83999999999997 127.0 0) (effects (font (size 1 1)) hide))
-              (property "MPN" "MSPM0L1105TRHBR" (at 243.83999999999997 127.0 0) (effects (font (size 1 1)) hide))
+              (property "MPN" "MSPM0L1106TRHBR" (at 243.83999999999997 127.0 0) (effects (font (size 1 1)) hide))
               (instances (project "groundlark-daqhat-01" (path "/de5c43d7-546f-5b4d-b587-d8dfceb38170/f6bfc69a-2b11-5d7b-82d1-e99b72f3d077" (reference "U130") (unit 1)))))
 (no_connect (at 228.6 106.68))
