File: hw/burrowlark-usb/boards/groundlark-field-head/03-sensors-page-01.kicad_sch (KiCad schematic)
At the start: 9 parts, among them U2 RM3100 XYZ, U3 DLVR-F50D option, U5 TPS22919

Commit message: Remove Burrowlark infrasound hardware and refresh board previews
Keep DAQUSB-01 magnetometer-only across the circuit, routed PCB, BOM, review schematic and native routing snapshot. Publish the refreshed render in the main README and add population regression checks.

Validation: 125 pin checks, clean ERC/DRC, native routing replay, 3 Burrowlark regression tests and lab unit tests pass. Full lab builds pass; hardware regressions stop on unrelated DAQHAT-01 assembly registry/source mismatches.
Parts:
- removed C5: 100n, Groundlark:Capacitor_SMD__C_0603_1608Metric, symbol Groundlark:Part_C5
- removed U3: DLVR-F50D option, Groundlark:Groundlark__DLVR_E1BS, symbol Groundlark:Part_U3
Changed lines of the file:
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@@
               (property "Footprint" "Groundlark:Package_TO_SOT_SMD__SOT-363_SC-70-6" (at 45.72 40.64 0) (effects (font (size 1 1)) hide))
               (property "MPN" "TPS22919DCKR" (at 45.72 40.64 0) (effects (font (size 1 1)) hide))
-              (instances (project "groundlark-field-head" (path "/3e18d740-4de4-5e4c-8150-31b96f65f152/7bec89a2-520f-51ab-8226-ae13c36b967f" (reference "U5") (unit 1)))))
+              (instances (project "groundlark-field-head" (path "/e1043b90-5a3a-5d7b-9b91-8488ec3f38a4/ab979e54-c171-5922-9bbc-4aaabc504545" (reference "U5") (unit 1)))))
 (wire (pts (xy 30.48 38.1) (xy 25.4 38.1)) (stroke (width 0) (type default)))
 (global_label "V3" (shape bidirectional) (at 25.4 38.1 180) (effects (font (size 0.9 0.9)) (justify right)))
@@
               (property "Footprint" "Groundlark:Resistor_SMD__R_0603_1608Metric" (at 142.24 38.1 0) (effects (font (size 1 1)) hide))
               (property "MPN" "RC0603FR-07100KL" (at 142.24 38.1 0) (effects (font (size 1 1)) hide))
-              (instances (project "groundlark-field-head" (path "/3e18d740-4de4-5e4c-8150-31b96f65f152/7bec89a2-520f-51ab-8226-ae13c36b967f" (reference "R5") (unit 1)))))
+              (instances (project "groundlark-field-head" (path "/e1043b90-5a3a-5d7b-9b91-8488ec3f38a4/ab979e54-c171-5922-9bbc-4aaabc504545" (reference "R5") (unit 1)))))
 (wire (pts (xy 127.0 38.1) (xy 121.92 38.1)) (stroke (width 0) (type default)))
 (global_label "SENSOR_EN" (shape bidirectional) (at 121.92 38.1 180) (effects (font (size 0.9 0.9)) (justify right)))
@@
               (property "Footprint" "Groundlark:Capacitor_SMD__C_0603_1608Metric" (at 238.76 38.1 0) (effects (font (size 1 1)) hide))
               (property "MPN" "GRM188R71H104KA93D" (at 238.76 38.1 0) (effects (font (size 1 1)) hide))
-              (instances (project "groundlark-field-head" (path "/3e18d740-4de4-5e4c-8150-31b96f65f152/7bec89a2-520f-51ab-8226-ae13c36b967f" (reference "C9") (unit 1)))))
+              (instances (project "groundlark-field-head" (path "/e1043b90-5a3a-5d7b-9b91-8488ec3f38a4/ab979e54-c171-5922-9bbc-4aaabc504545" (reference "C9") (unit 1)))))
 (wire (pts (xy 223.52 38.1) (xy 218.44 38.1)) (stroke (width 0) (type default)))
 (global_label "V3" (shape bidirectional) (at 218.44 38.1 180) (effects (font (size 0.9 0.9)) (justify right)))
@@
               (property "Footprint" "Groundlark:Resistor_SMD__R_0603_1608Metric" (at 335.28 38.1 0) (effects (font (size 1 1)) hide))
               (property "MPN" "RC0603FR-074K7L" (at 335.28 38.1 0) (effects (font (size 1 1)) hide))
-              (instances (project "groundlark-field-head" (path "/3e18d740-4de4-5e4c-8150-31b96f65f152/7bec89a2-520f-51ab-8226-ae13c36b967f" (reference "R7") (unit 1)))))
+              (instances (project "groundlark-field-head" (path "/e1043b90-5a3a-5d7b-9b91-8488ec3f38a4/ab979e54-c171-5922-9bbc-4aaabc504545" (reference "R7") (unit 1)))))
 (wire (pts (xy 320.04 38.1) (xy 314.96 38.1)) (stroke (width 0) (type default)))
 (global_label "SDA" (shape bidirectional) (at 314.96 38.1 180) (effects (font (size 0.9 0.9)) (justify right)))
@@
               (property "Footprint" "Groundlark:Resistor_SMD__R_0603_1608Metric" (at 45.72 71.12 0) (effects (font (size 1 1)) hide))
               (property "MPN" "RC0603FR-074K7L" (at 45.72 71.12 0) (effects (font (size 1 1)) hide))
-              (instances (project "groundlark-field-head" (path "/3e18d740-4de4-5e4c-8150-31b96f65f152/7bec89a2-520f-51ab-8226-ae13c36b967f" (reference "R8") (unit 1)))))
+              (instances (project "groundlark-field-head" (path "/e1043b90-5a3a-5d7b-9b91-8488ec3f38a4/ab979e54-c171-5922-9bbc-4aaabc504545" (reference "R8") (unit 1)))))
 (wire (pts (xy 30.48 71.12) (xy 25.4 71.12)) (stroke (width 0) (type default)))
 (global_label "SCL" (shape bidirectional) (at 25.4 71.12 180) (effects (font (size 0.9 0.9)) (justify right)))
@@
               (property "Footprint" "Groundlark:Groundlark__PNI_14190_Module" (at 142.24 78.74 0) (effects (font (size 1 1)) hide))
               (property "MPN" "PNI 14190" (at 142.24 78.74 0) (effects (font (size 1 1)) hide))
-              (instances (project "groundlark-field-head" (path "/3e18d740-4de4-5e4c-8150-31b96f65f152/7bec89a2-520f-51ab-8226-ae13c36b967f" (reference "U2") (unit 1)))))
+              (instances (project "groundlark-field-head" (path "/e1043b90-5a3a-5d7b-9b91-8488ec3f38a4/ab979e54-c171-5922-9bbc-4aaabc504545" (reference "U2") (unit 1)))))
 (wire (pts (xy 127.0 71.12) (xy 121.92 71.12)) (stroke (width 0) (type default)))
 (global_label "SCL" (shape bidirectional) (at 121.92 71.12 180) (effects (font (size 0.9 0.9)) (justify right)))
@@
               (property "Footprint" "Groundlark:Capacitor_SMD__C_0603_1608Metric" (at 238.76 71.12 0) (effects (font (size 1 1)) hide))
               (property "MPN" "GRM188R71H104KA93D" (at 238.76 71.12 0) (effects (font (size 1 1)) hide))
-              (instances (project "groundlark-field-head" (path "/3e18d740-4de4-5e4c-8150-31b96f65f152/7bec89a2-520f-51ab-8226-ae13c36b967f" (reference "C4") (unit 1)))))
+              (instances (project "groundlark-field-head" (path "/e1043b90-5a3a-5d7b-9b91-8488ec3f38a4/ab979e54-c171-5922-9bbc-4aaabc504545" (reference "C4") (unit 1)))))
 (wire (pts (xy 223.52 71.12) (xy 218.44 71.12)) (stroke (width 0) (type default)))
 (global_label "V3_SENSOR" (shape bidirectional) (at 218.44 71.12 180) (effects (font (size 0.9 0.9)) (justify right)))
 (wire (pts (xy 254.0 71.12) (xy 259.08 71.12)) (stroke (width 0) (type default)))
 (global_label "GND" (shape bidirectional) (at 259.08 71.12 0) (effects (font (size 0.9 0.9)) (justify left)))
-(symbol (lib_id "Groundlark:Part_U3") (at 335.28 72.39 0) (unit 1) (in_bom yes) (on_board yes) (dnp yes)
-              (property "Reference" "U3" (at 335.28 64.58 0) (effects (font (size 1.27 1.27))))
-              (property "Value" "DLVR-F50D option" (at 335.28 67.08 0) (effects (font (size 1.0 1.0))))
-              (property "Footprint" "Groundlark:Groundlark__DLVR_E1BS" (at 335.28 72.39 0) (effects (font (size 1 1)) hide))
-              (property "MPN" "DLVR-F50D-E1BS-I-NI3F" (at 335.28 72.39 0) (effects (font (size 1 1)) hide))
-              (instances (project "groundlark-field-head" (path "/3e18d740-4de4-5e4c-8150-31b96f65f152/7bec89a2-520f-51ab-8226-ae13c36b967f" (reference "U3") (unit 1)))))
-(wire (pts (xy 320.04 71.12) (xy 314.96 71.12)) (stroke (width 0) (type default)))
-(global_label "GND" (shape bidirectional) (at 314.96 71.12 180) (effects (font (size 0.9 0.9)) (justify right)))
-(wire (pts (xy 320.04 73.66) (xy 314.96 73.66)) (stroke (width 0) (type default)))
-(global_label "V3_SENSOR" (shape bidirectional) (at 314.96 73.66 180) (effects (font (size 0.9 0.9)) (justify right)))
-(wire (pts (xy 350.52 71.12) (xy 355.6 71.12)) (stroke (width 0) (type default)))
-(global_label "SDA" (shape bidirectional) (at 355.6 71.12 0) (effects (font (size 0.9 0.9)) (justify left)))
-(wire (pts (xy 350.52 73.66) (xy 355.6 73.66)) (stroke (width 0) (type default)))
-(global_label "SCL" (shape bidirectional) (at 355.6 73.66 0) (effects (font (size 0.9 0.9)) (justify left)))
-(symbol (lib_id "Groundlark:Part_C5") (at 45.72 114.3 0) (unit 1) (in_bom yes) (on_board yes) (dnp no)
-              (property "Reference" "C5" (at 45.72 107.75999999999999 0) (effects (font (size 1.27 1.27))))
-              (property "Value" "100n" (at 45.72 110.25999999999999 0) (effects (font (size 1.0 1.0))))
-              (property "Footprint" "Groundlark:Capacitor_SMD__C_0603_1608Metric" (at 45.72 114.3 0) (effects (font (size 1 1)) hide))
-              (property "MPN" "GRM188R71H104KA93D" (at 45.72 114.3 0) (effects (font (size 1 1)) hide))
-              (instances (project "groundlark-field-head" (path "/3e18d740-4de4-5e4c-8150-31b96f65f152/7bec89a2-520f-51ab-8226-ae13c36b967f" (reference "C5") (unit 1)))))
-(wire (pts (xy 30.48 114.3) (xy 25.4 114.3)) (stroke (width 0) (type default)))
-(global_label "V3_SENSOR" (shape bidirectional) (at 25.4 114.3 180) (effects (font (size 0.9 0.9)) (justify right)))
-(wire (pts (xy 60.96 114.3) (xy 66.04 114.3)) (stroke (width 0) (type default)))
-(global_label "GND" (shape bidirectional) (at 66.04 114.3 0) (effects (font (size 0.9 0.9)) (justify left)))
 )

Commit message: Add SHT45 enclosure climate sensing to Burrowlark
Add Sensirion SHT45-AD1B-R2 U6 and switched-rail bypass C10, with JLCPCB C5221601 stock evidence. Synchronize circuit, routed PCB, native SES, schematic, BOM, README render and browser model.

Publish CRC-checked raw climate sensor 17 through simulation, recording and replay. Add enclosure controls, independent fault/recovery checks and protocol fixtures. The isolated software profile passes 213 tests; Burrowlark DRC/ERC and copper replay pass. Full hardware regression remains blocked by pre-existing assembly registry mismatches. MCU firmware and physical qualification remain pending.
Parts:
- added C10: 100n, Groundlark:Capacitor_SMD__C_0603_1608Metric, symbol Groundlark:Part_C10
- added U6: SHT45, Groundlark:SHT45, symbol Groundlark:Part_U6
Connections:
- net GND: now also C10.2, U6.4 (VSS)
- net SCL: now also U6.2 (SCL)
- net SDA: now also U6.1 (SDA)
- net V3_SENSOR: now also C10.1, U6.3 (VDD)
Changed lines of the file:
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@@
 (wire (pts (xy 254.0 71.12) (xy 259.08 71.12)) (stroke (width 0) (type default)))
 (global_label "GND" (shape bidirectional) (at 259.08 71.12 0) (effects (font (size 0.9 0.9)) (justify left)))
+(symbol (lib_id "Groundlark:Part_U6") (at 335.28 72.39 0) (unit 1) (in_bom yes) (on_board yes) (dnp no)
+              (property "Reference" "U6" (at 335.28 64.58 0) (effects (font (size 1.27 1.27))))
+              (property "Value" "SHT45" (at 335.28 67.08 0) (effects (font (size 1.0 1.0))))
+              (property "Footprint" "Groundlark:SHT45" (at 335.28 72.39 0) (effects (font (size 1 1)) hide))
+              (property "MPN" "SHT45-AD1B-R2" (at 335.28 72.39 0) (effects (font (size 1 1)) hide))
+              (instances (project "groundlark-field-head" (path "/e1043b90-5a3a-5d7b-9b91-8488ec3f38a4/ab979e54-c171-5922-9bbc-4aaabc504545" (reference "U6") (unit 1)))))
+(wire (pts (xy 320.04 71.12) (xy 314.96 71.12)) (stroke (width 0) (type default)))
+(global_label "SDA" (shape bidirectional) (at 314.96 71.12 180) (effects (font (size 0.9 0.9)) (justify right)))
+(wire (pts (xy 320.04 73.66) (xy 314.96 73.66)) (stroke (width 0) (type default)))
+(global_label "SCL" (shape bidirectional) (at 314.96 73.66 180) (effects (font (size 0.9 0.9)) (justify right)))
+(wire (pts (xy 350.52 71.12) (xy 355.6 71.12)) (stroke (width 0) (type default)))
+(global_label "V3_SENSOR" (shape bidirectional) (at 355.6 71.12 0) (effects (font (size 0.9 0.9)) (justify left)))
+(wire (pts (xy 350.52 73.66) (xy 355.6 73.66)) (stroke (width 0) (type default)))
+(global_label "GND" (shape bidirectional) (at 355.6 73.66 0) (effects (font (size 0.9 0.9)) (justify left)))
+(symbol (lib_id "Groundlark:Part_C10") (at 45.72 114.3 0) (unit 1) (in_bom yes) (on_board yes) (dnp no)
+              (property "Reference" "C10" (at 45.72 107.75999999999999 0) (effects (font (size 1.27 1.27))))
+              (property "Value" "100n" (at 45.72 110.25999999999999 0) (effects (font (size 1.0 1.0))))
+              (property "Footprint" "Groundlark:Capacitor_SMD__C_0603_1608Metric" (at 45.72 114.3 0) (effects (font (size 1 1)) hide))
+              (property "MPN" "GRM188R71H104KA93D" (at 45.72 114.3 0) (effects (font (size 1 1)) hide))
+              (instances (project "groundlark-field-head" (path "/e1043b90-5a3a-5d7b-9b91-8488ec3f38a4/ab979e54-c171-5922-9bbc-4aaabc504545" (reference "C10") (unit 1)))))
+(wire (pts (xy 30.48 114.3) (xy 25.4 114.3)) (stroke (width 0) (type default)))
+(global_label "V3_SENSOR" (shape bidirectional) (at 25.4 114.3 180) (effects (font (size 0.9 0.9)) (justify right)))
+(wire (pts (xy 60.96 114.3) (xy 66.04 114.3)) (stroke (width 0) (type default)))
+(global_label "GND" (shape bidirectional) (at 66.04 114.3 0) (effects (font (size 0.9 0.9)) (justify left)))
 )
