File: hw/burrowlark-usb/boards/groundlark-field-head/groundlark-field-head.kicad_pcb (KiCad board)
At the start: 4 copper layers, 70 x 45 mm, 31 parts, among them J1 USB-C DEVICE, J2 SWD / 3V3 SENSE, J3 BOOT0 jumper, U1 STM32F042K6T6, U2 RM3100 XYZ, U3 DLVR-F50D option, U4 AP2112K-3.3, U5 TPS22919

Commit message: Remove Burrowlark infrasound hardware and refresh board previews
Keep DAQUSB-01 magnetometer-only across the circuit, routed PCB, BOM, review schematic and native routing snapshot. Publish the refreshed render in the main README and add population regression checks.

Validation: 125 pin checks, clean ERC/DRC, native routing replay, 3 Burrowlark regression tests and lab unit tests pass. Full lab builds pass; hardware regressions stop on unrelated DAQHAT-01 assembly registry/source mismatches.
Parts:
- removed C5: 100n, Groundlark:Capacitor_SMD__C_0603_1608Metric
- removed U3: DLVR-F50D option, Groundlark:Groundlark__DLVR_E1BS
Routing:
- net GND: track 250.6 -> 209.5 mm, vias 1 -> 2
- net SCL: track 78.9 -> 54.6 mm, vias 1 -> 0
- net SDA: track 72.1 -> 49.7 mm

Commit message: Add SHT45 enclosure climate sensing to Burrowlark
Add Sensirion SHT45-AD1B-R2 U6 and switched-rail bypass C10, with JLCPCB C5221601 stock evidence. Synchronize circuit, routed PCB, native SES, schematic, BOM, README render and browser model.

Publish CRC-checked raw climate sensor 17 through simulation, recording and replay. Add enclosure controls, independent fault/recovery checks and protocol fixtures. The isolated software profile passes 213 tests; Burrowlark DRC/ERC and copper replay pass. Full hardware regression remains blocked by pre-existing assembly registry mismatches. MCU firmware and physical qualification remain pending.
Parts:
- added C10: 100n, Groundlark:Capacitor_SMD__C_0603_1608Metric, F.Cu at (83.0, 88.0)
- added U6: SHT45, Groundlark:SHT45, F.Cu at (81.0, 86.0)
Routing:
- net SCL: track 54.6 -> 91.4 mm, vias 0 -> 4
- net SDA: track 49.7 -> 79.8 mm, vias 2 -> 4
- net V3_SENSOR: track 64.7 -> 72.8 mm
- net GND: track 209.5 -> 210.9 mm, vias 2 -> 4
Other:
- board text added: "Burrowlark DAQUSB-01"
- board text removed: "Groundlark FIELD A2"

Commit message: Add Burrowlark favicon and revision silkscreen
Place the shared favicon above the Burrowlark name and DAQUSB-01 / REV A2 label. Preserve the existing A2 revision and all 579 tracks/vias; author the artwork in placement metadata and retain it on assembly regeneration.

Refresh README render, board previews and browser model/provenance. Native DRC/ERC, copper replay, repository structure, lab unit tests and workbench HTTP/browser checks pass.
Other:
- board text added: "Burrowlark"
- board text added: "DAQUSB-01 / REV A2"
- board text removed: "Burrowlark DAQUSB-01"
