File: hw/skylark-usb/layout/skylark/skylark.kicad_pcb (KiCad board)
At the start: 2 copper layers, 117 parts

Commit message: Harden Skylark signal chain and add manufacturing audit
Parts:
- added C80: , skylark:Capacitor_SMD__C_1206_3216Metric, F.Cu at (20.0, 0.00)
- added C81: , skylark:Capacitor_SMD__C_1206_3216Metric, F.Cu at (30.0, 0.00)
- added C82: , skylark:Capacitor_SMD__C_1206_3216Metric, F.Cu at (40.0, 0.00)
- added C83: , skylark:Capacitor_SMD__C_1206_3216Metric, F.Cu at (50.0, 0.00)
- added C84: , skylark:Capacitor_SMD__C_1206_3216Metric, F.Cu at (60.0, 0.00)
- added C85: , skylark:Capacitor_SMD__C_1206_3216Metric, F.Cu at (70.0, 0.00)
- added C86: , skylark:Capacitor_SMD__C_1206_3216Metric, F.Cu at (80.0, 0.00)
- added C87: , skylark:Capacitor_SMD__C_1206_3216Metric, F.Cu at (90.0, 0.00)
- added D4: , skylark:Package_TO_SOT_SMD__SOT-23, F.Cu at (10.0, 0.00)
- added R74, R75: , skylark:Resistor_SMD__R_0603_1608Metric, F.Cu at (0.00, 0.00)
- C30, C33, C36, C50, C53, C56: footprint skylark:Capacitor_SMD__C_0603_1608Metric -> skylark:Capacitor_SMD__C_1206_3216Metric
Connections:
- net 2 renamed u1-2
- Q7 pad 1: CLAMP_HOLD -> CLAMP_BASE
- Q7 pad 2: GND -> VZERO
- R70 pad 1: USB_5V -> GATE_SUPPLY
- R71 pad 2: GND -> VZERO

Commit message: Finalize Skylark signal-chain updates and remove obsolete artifacts
Parts:
- C31, C34, C51, C54: value (none) -> 10uF; footprint skylark:Capacitor_SMD__C_0603_1608Metric -> Skylark:Capacitor_SMD__C_0805_2012Metric
- J1: value (none) -> TYPE-C-31-M-12; footprint skylark:Connector_USB__USB_C_Receptacle_GCT_USB4105-xx-A_16P_TopMnt_Horizontal -> Skylark:USB_C_HRO_TYPE-C-31-M-12
- R3: value (none) -> 82000R; footprint skylark:Resistor_SMD__R_0603_1608Metric -> Skylark:Resistor_SMD__R_0603_1608Metric
- U12: value (none) -> BMP388; footprint skylark:BMP390 -> Skylark:BMP388
